File: MultiplexadorSerial/sch/MultiplexadorSerial.kicad_pcb (KiCad board)
At the start: 2 copper layers, 69.2 x 54 mm, 65 parts, among them J1 SL4, J2 SL3, J3 SL1, J4 SL2, Q1 Q_NPN_CBE, Q2 Q_NPN_CBE, Q3 Q_NPN_CBE, Q4 Q_NPN_CBE, U1 SP3481CP, U2 SP3481CP, U3 SP3481CP, U4 SP3481CP, U5 4052

Commit message: Signed-off-by: cuki2 <mauricio@krebs.com.br>
Parts:
- moved U1 97.1 mm to (121.5, 66.3)
- moved J1 97.1 mm to (121.7, 58.3)
- moved J2 84.5 mm to (105.4, 89.9)
- moved U2 66.7 mm to (148.8, 56.3)
- moved Q2 66.7 mm to (141.7, 57.9)
- moved C1 47.8 mm to (105.3, 84.4)
- moved C2 47.8 mm to (105.3, 84.4)
- moved C5 47.8 mm to (105.3, 84.4)
- moved Q1 47.8 mm to (105.3, 84.4)
- moved R1 47.8 mm to (105.3, 84.4)
- moved R10 47.8 mm to (105.3, 84.4)
- moved R11 47.8 mm to (105.3, 84.4)
- moved R12 47.8 mm to (105.3, 84.4)
- moved R13 47.8 mm to (105.3, 84.4)
- moved R14 47.8 mm to (105.3, 84.4)
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Changed lines of the file:
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@@
   (general
     (links 133)
-    (no_connects 103)
+    (no_connects 100)
     (area 99.619999 46.279999 168.985001 100.405001)
     (thickness 1.6)
@@
   )
   (module w_smd_cap:c_0805 (layer F.Cu)
-    (at 148.5011 105.0036)
+    (at 105.3211 84.4296)
     (descr "SMT capacitor, 0805")
     (fp_text reference C1 (at 0 -0.9906) (layer F.SilkS)
@@
   )
   (module w_smd_cap:c_0805 (layer F.Cu)
-    (at 148.5011 105.0036)
+    (at 105.3211 84.4296)
     (descr "SMT capacitor, 0805")
     (fp_text reference C2 (at 0 -0.9906) (layer F.SilkS)
@@
   )
   (module w_smd_cap:c_0805 (layer F.Cu)
-    (at 148.5011 105.0036)
+    (at 105.3211 84.4296)
     (descr "SMT capacitor, 0805")
     (fp_text reference C5 (at 0 -0.9906) (layer F.SilkS)
@@
   )
   (module w_pin_strip:pin_socket_2 (layer F.Cu)
-    (at 32.258 20.447 180)
+    (at 121.666 58.293 180)
     (descr "Pin socket 2pin")
     (tags "CONN DEV")
@@
   )
   (module w_pin_strip:pin_socket_2 (layer F.Cu)
-    (at 32.131 47.879 180)
+    (at 105.41 89.916 180)
     (descr "Pin socket 2pin")
     (tags "CONN DEV")
@@
   )
   (module w_smd_trans:sot23 (layer F.Cu)
-    (at 148.5011 105.0036)
+    (at 105.3211 84.4296)
     (descr SOT23)
     (fp_text reference Q1 (at 0.0254 -0.3302) (layer F.SilkS)
@@
   )
   (module w_smd_resistors:r_0805 (layer F.Cu)
-    (at 148.5011 105.0036)
+    (at 105.3211 84.4296)
     (descr "SMT resistor, 0805")
     (fp_text reference R1 (at 0 -0.9906) (layer F.SilkS)
@@
   )
   (module w_smd_resistors:r_0805 (layer F.Cu)
-    (at 148.5011 105.0036)
+    (at 105.3211 84.4296)
     (descr "SMT resistor, 0805")
     (fp_text reference R2 (at 0 -0.9906) (layer F.SilkS)
@@
   )
   (module w_smd_resistors:r_0805 (layer F.Cu)
-    (at 148.5011 105.0036)
+    (at 105.3211 84.4296)
     (descr "SMT resistor, 0805")
     (fp_text reference R3 (at 0 -0.9906) (layer F.SilkS)
@@
   )
   (module w_smd_resistors:r_0805 (layer F.Cu)
-    (at 148.5011 105.0036)
+    (at 105.3211 84.4296)
     (descr "SMT resistor, 0805")
     (fp_text reference R4 (at 0 -0.9906) (layer F.SilkS)
@@
   )
   (module w_smd_resistors:r_0805 (layer F.Cu)
-    (at 148.5011 105.0036)
+    (at 105.3211 84.4296)
     (descr "SMT resistor, 0805")
     (fp_text reference R5 (at 0 -0.9906) (layer F.SilkS)
@@
   )
   (module w_smd_resistors:r_0805 (layer F.Cu)
-    (at 148.5011 105.0036)
+    (at 105.3211 84.4296)
     (descr "SMT resistor, 0805")
     (fp_text reference R6 (at 0 -0.9906) (layer F.SilkS)
@@
   )
   (module w_smd_resistors:r_0805 (layer F.Cu)
-    (at 148.5011 105.0036)
+    (at 105.3211 84.4296)
     (descr "SMT resistor, 0805")
     (fp_text reference R7 (at 0 -0.9906) (layer F.SilkS)
@@
   )
   (module w_smd_resistors:r_0805 (layer F.Cu)
-    (at 148.5011 105.0036)
+    (at 105.3211 84.4296)
     (descr "SMT resistor, 0805")
     (fp_text reference R8 (at 0 -0.9906) (layer F.SilkS)
@@
   )
   (module w_smd_resistors:r_0805 (layer F.Cu)
-    (at 148.5011 105.0036)
+    (at 105.3211 84.4296)
     (descr "SMT resistor, 0805")
     (fp_text reference R9 (at 0 -0.9906) (layer F.SilkS)
@@
   )
   (module w_smd_resistors:r_0805 (layer F.Cu)
-    (at 148.5011 105.0036)
+    (at 105.3211 84.4296)
     (descr "SMT resistor, 0805")
     (fp_text reference R10 (at 0 -0.9906) (layer F.SilkS)
@@
   )
   (module w_smd_resistors:r_0805 (layer F.Cu)
-    (at 148.5011 105.0036)
+    (at 105.3211 84.4296)
     (descr "SMT resistor, 0805")
     (fp_text reference R11 (at 0 -0.9906) (layer F.SilkS)
@@
   )
   (module w_smd_resistors:r_0805 (layer F.Cu)
-    (at 148.5011 105.0036)
+    (at 105.3211 84.4296)
     (descr "SMT resistor, 0805")
     (fp_text reference R12 (at 0 -0.9906) (layer F.SilkS)
@@
   )
   (module w_smd_resistors:r_0805 (layer F.Cu)
-    (at 148.5011 105.0036)
+    (at 105.3211 84.4296)
     (descr "SMT resistor, 0805")
     (fp_text reference R13 (at 0 -0.9906) (layer F.SilkS)
@@
   )
   (module w_smd_resistors:r_0805 (layer F.Cu)
-    (at 148.5011 105.0036)
+    (at 105.3211 84.4296)
     (descr "SMT resistor, 0805")
     (fp_text reference R14 (at 0 -0.9906) (layer F.SilkS)
@@
   )
   (module w_smd_resistors:r_0805 (layer F.Cu)
-    (at 148.5011 105.0036)
+    (at 105.3211 84.4296)
     (descr "SMT resistor, 0805")
     (fp_text reference R15 (at 0 -0.9906) (layer F.SilkS)
@@
   )
   (module w_smd_resistors:r_0805 (layer F.Cu)
-    (at 148.5011 105.0036)
+    (at 105.3211 84.4296)
     (descr "SMT resistor, 0805")
     (fp_text reference R16 (at 0 -0.9906) (layer F.SilkS)
@@
   )
   (module w_smd_resistors:r_0805 (layer F.Cu)
-    (at 148.5011 105.0036)
+    (at 105.3211 84.4296)
     (descr "SMT resistor, 0805")
     (fp_text reference R35 (at 0 -0.9906) (layer F.SilkS)
@@
   )
   (module w_smd_resistors:r_0805 (layer F.Cu)
-    (at 148.5011 105.0036)
+    (at 105.3211 84.4296)
     (descr "SMT resistor, 0805")
     (fp_text reference R40 (at 0 -0.9906) (layer F.SilkS)
@@
   )
   (module w_smd_resistors:r_0805 (layer F.Cu)
-    (at 148.5011 105.0036)
+    (at 105.3211 84.4296)
     (descr "SMT resistor, 0805")
     (fp_text reference R41 (at 0 -0.9906) (layer F.SilkS)
@@
   )
   (module w_smd_resistors:r_0805 (layer F.Cu)
-    (at 148.5011 105.0036)
+    (at 105.3211 84.4296)
     (descr "SMT resistor, 0805")
     (fp_text reference R42 (at 0 -0.9906) (layer F.SilkS)
@@
   )
   (module w_smd_dil:so-8 (layer F.Cu)
-    (at 32.131 28.448)
+    (at 121.539 66.294)
     (descr SO-8)
     (fp_text reference U1 (at 0 -1.016) (layer F.SilkS)
@@
   )
   (module w_smd_dil:so-8 (layer F.Cu)
-    (at 214.122 69.723 270)
+    (at 148.844 56.261 270)
     (descr SO-8)
     (fp_text reference U2 (at 0 -0.127 270) (layer F.SilkS)
@@
   )
   (module w_smd_trans:sot23 (layer F.Cu)
-    (at 207.01 71.374 90)
+    (at 141.732 57.912 90)
     (descr SOT23)
     (fp_text reference Q2 (at 0 0.127 90) (layer F.SilkS)
