File: MultiplexadorSerial/sch/MultiplexadorSerial.kicad_pcb (KiCad board)
At the start: 2 copper layers, 69.2 x 54 mm, 65 parts, among them J1 SL4, J2 SL3, J3 SL1, J4 SL2, Q1 Q_NPN_CBE, Q2 Q_NPN_CBE, Q3 Q_NPN_CBE, Q4 Q_NPN_CBE, U1 SP3481CP, U2 SP3481CP, U3 SP3481CP, U4 SP3481CP, U5 4052

Commit message: novo desenho
Signed-off-by: cuki2 <mauricio@krebs.com.br>
Parts:
- added J5: SL4, w_pin_strip:pin_socket_2, F.Cu at (160.3, 87.6)
- added R44, R45: 560R, w_smd_resistors:r_0805, F.Cu at (181.8, 68.4)
- D1: value PWR -> TX
- D2: value TX -> PWR
- J1: value SL4 -> SL; footprint w_pin_strip:pin_socket_2 -> w_pin_strip:pin_socket_3
- J2: value SL3 -> SL1
- J3: value SL1 -> SL2
- J4: value SL2 -> SL3
- R1, R2: value 10k -> 1k2
- R10, R18, R26: value 10k -> 560R
- R11, R27: value 120R -> 560R
- R12, R16: value 560R -> 330R
- R13: value 120R -> 330R
- R14, R15, R19, R20, R24, R28, R3, R30, R39, R4, R8: value 560R -> 10k
- R17: value 10k -> 330R
- R22, R40, R41, R6: value 10k -> 360R
- R23, R31, R32, R7: value 560R -> 360R
- R25, R43, R9: value 10k -> 120R
- R29: value 120R -> 10k
- R33, R37: value 1k2 -> 10k
- R34: value 330R -> 120R
- R35, R36: value 330R -> 560R
- R38: value 330R -> 10k
- U2: value SP3481CP -> 4052; footprint w_smd_dil:so-8 -> w_smd_dil:so-16
- U5: value 4052 -> SP3481CP; footprint w_smd_dil:so-16 -> w_smd_dil:so-8
- moved J1 87.1 mm to (208.8, 59.9), turned to 0 degrees
- moved J2 82.4 mm to (187.5, 82.5), turned to 0 degrees
- moved C1 78.1 mm to (181.8, 68.4)
- moved C2 78.1 mm to (181.8, 68.4)
- moved C5 78.1 mm to (181.8, 68.4)
- moved Q1 78.1 mm to (181.8, 68.4)
- moved R1 78.1 mm to (181.8, 68.4)
- moved R10 78.1 mm to (181.8, 68.4)
- moved R11 78.1 mm to (181.8, 68.4)
- moved R12 78.1 mm to (181.8, 68.4)
- moved R13 78.1 mm to (181.8, 68.4)
- moved R14 78.1 mm to (181.8, 68.4)
- moved R15 78.1 mm to (181.8, 68.4)
- moved R16 78.1 mm to (181.8, 68.4)
- moved R2 78.1 mm to (181.8, 68.4)
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Connections:
- C1 pad 1: VDD -> +5V
- C2 pad 1: VDD -> +5V
- C3 pad 1: VDD -> +5V
- C4 pad 1: VDD -> +5V
- C5 pad 1: VDD -> +5V
- D1 pad 1: VDD -> Net-(D1-Pad1)
- D1 pad 2: Net-(D1-Pad2) -> /TX
- D2 pad 1: Net-(D2-Pad1) -> +5V
- J1 pad 1: Net-(J1-Pad1) -> /TX
- J1 pad 2: Net-(J1-Pad2) -> /RX
- R1 pad 1: Net-(Q1-Pad2) -> +5V
- R1 pad 2: Net-(R1-Pad2) -> Net-(D1-Pad1)
- R10 pad 1: Net-(R10-Pad1) -> Net-(J2-Pad2)
- R10 pad 2: VDD -> GND
- R11 pad 1: Net-(J1-Pad1) -> +5V
- R11 pad 2: Net-(J1-Pad2) -> Net-(J2-Pad1)
- R12 pad 1: Net-(J1-Pad2) -> /ADR0
- R12 pad 2: GND -> Net-(R12-Pad2)
- R13 pad 1: Net-(J2-Pad1) -> /ADR1
- R13 pad 2: Net-(J2-Pad2) -> Net-(R13-Pad2)
- R14 pad 1: Net-(J2-Pad2) -> GND
- R14 pad 2: GND -> Net-(R12-Pad2)
- R15 pad 1: VDD -> GND
- R15 pad 2: Net-(J1-Pad1) -> Net-(R13-Pad2)
- R16 pad 1: VDD -> /TX
- R16 pad 2: Net-(J2-Pad1) -> Net-(R16-Pad2)
- R17 pad 1: Net-(Q3-Pad2) -> /RX
- R17 pad 2: Net-(R17-Pad2) -> Net-(D3-Pad2)
- R18 pad 1: Net-(Q4-Pad2) -> +5V
- R18 pad 2: Net-(R18-Pad2) -> Net-(D3-Pad1)
- R19 pad 1: Net-(R17-Pad2) -> Net-(Q2-Pad2)
- R19 pad 2: Net-(R19-Pad2) -> /RX2
- R2 pad 1: Net-(Q2-Pad2) -> GND
- R2 pad 2: Net-(R2-Pad2) -> Net-(D2-Pad2)
- R20 pad 1: Net-(R18-Pad2) -> +5V
- R20 pad 2: Net-(R20-Pad2) -> Net-(Q2-Pad3)
- R21 pad 1: VDD -> /TX2
- R21 pad 2: Net-(Q3-Pad3) -> +5V
- R22 pad 1: VDD -> /RX2
- R22 pad 2: Net-(Q4-Pad3) -> Net-(R22-Pad2)
- R23 pad 1: Net-(R23-Pad1) -> /TX2
- R24 pad 1: Net-(R24-Pad1) -> +5V
- R24 pad 2: Net-(R24-Pad2) -> Net-(R22-Pad2)
- R25 pad 1: Net-(R19-Pad2) -> Net-(J3-Pad1)
- R25 pad 2: VDD -> Net-(J3-Pad2)
- R26 pad 1: Net-(R20-Pad2) -> Net-(J3-Pad2)
- R26 pad 2: VDD -> GND
- R27 pad 1: Net-(J3-Pad1) -> +5V
- R27 pad 2: Net-(J3-Pad2) -> Net-(J3-Pad1)
- R28 pad 1: Net-(J3-Pad2) -> Net-(Q3-Pad2)
- R28 pad 2: GND -> /RX3
- R29 pad 1: Net-(J4-Pad1) -> +5V
- R29 pad 2: Net-(J4-Pad2) -> Net-(Q3-Pad3)
- R3 pad 1: Net-(R1-Pad2) -> Net-(Q1-Pad2)
- R3 pad 2: Net-(R3-Pad2) -> /RX1
- R30 pad 1: Net-(J4-Pad2) -> /TX3
- R30 pad 2: GND -> +5V
- R31 pad 1: VDD -> /RX3
- R31 pad 2: Net-(J3-Pad1) -> Net-(R31-Pad2)
- R32 pad 1: VDD -> /TX3
- R32 pad 2: Net-(J4-Pad1) -> Net-(R32-Pad2)
- R33 pad 1: Net-(D1-Pad2) -> +5V
- R33 pad 2: GND -> Net-(R31-Pad2)
- R34 pad 1: Net-(R34-Pad1) -> Net-(J4-Pad1)
- R34 pad 2: Net-(R34-Pad2) -> Net-(J4-Pad2)
- R35 pad 1: Net-(R35-Pad1) -> Net-(J4-Pad2)
- R35 pad 2: Net-(R35-Pad2) -> GND
- R36 pad 1: Net-(R36-Pad1) -> +5V
- R36 pad 2: Net-(D2-Pad2) -> Net-(J4-Pad1)
- R37 pad 1: VDD -> Net-(Q4-Pad2)
- R37 pad 2: Net-(D2-Pad1) -> /RX4
- R38 pad 1: Net-(D3-Pad2) -> +5V
- R38 pad 2: Net-(R38-Pad2) -> Net-(Q4-Pad3)
- R39 pad 1: VDD -> /TX4
- R39 pad 2: Net-(D3-Pad1) -> +5V
- R4 pad 1: Net-(R2-Pad2) -> +5V
- R4 pad 2: Net-(R10-Pad1) -> Net-(Q1-Pad3)
- R40 pad 1: VDD -> /RX4
- R41 pad 1: VDD -> /TX4
- R42 pad 1: VDD -> +5V
- R42 pad 2: Net-(R23-Pad2) -> Net-(R40-Pad2)
- R43 pad 1: VDD -> Net-(J5-Pad1)
- R43 pad 2: Net-(R24-Pad2) -> Net-(J5-Pad2)
- R5 pad 1: VDD -> /TX1
- R5 pad 2: Net-(Q1-Pad3) -> +5V
- R6 pad 1: VDD -> /RX1
- R6 pad 2: Net-(Q2-Pad3) -> Net-(R6-Pad2)
- R7 pad 1: Net-(R7-Pad1) -> /TX1
- R7 pad 2: Net-(R40-Pad2) -> Net-(R7-Pad2)
- R8 pad 1: Net-(R8-Pad1) -> +5V
- R8 pad 2: Net-(R41-Pad2) -> Net-(R6-Pad2)
- R9 pad 1: Net-(R3-Pad2) -> Net-(J2-Pad1)
- R9 pad 2: VDD -> Net-(J2-Pad2)
- SHIELD1 pad 0: Net-(D2-Pad2) -> /RX
- SHIELD1 pad 1: Net-(R38-Pad2) -> /TX
- SHIELD1 pad 5V: VDD -> +5V
- SHIELD1 pad AD0: Net-(R34-Pad2) -> /ADR0
- SHIELD1 pad AD1: Net-(R35-Pad2) -> /ADR1
- U1 pad 1: Net-(R40-Pad2) -> Net-(R6-Pad2)
- U1 pad 4: Net-(R3-Pad2) -> Net-(R7-Pad2)
- U1 pad 6: Net-(J1-Pad1) -> Net-(J2-Pad1)
- U1 pad 7: Net-(J1-Pad2) -> Net-(J2-Pad2)
- U1 pad 8: VDD -> +5V
- U2 pad 1: Net-(R41-Pad2) -> /RX1
- U2 pad 2: Net-(Q2-Pad3) -> /RX3
- U2 pad 3: Net-(Q2-Pad3) -> Net-(D3-Pad2)
- U2 pad 4: Net-(R10-Pad1) -> /RX4
- U2 pad 5: GND -> /RX2
- U2 pad 6: Net-(J2-Pad1) -> GND
- U2 pad 7: Net-(J2-Pad2) -> GND
- U2 pad 8: VDD -> GND
- U3 pad 1: Net-(R23-Pad2) -> Net-(R22-Pad2)
- U3 pad 2: Net-(Q3-Pad3) -> Net-(Q2-Pad3)
- U3 pad 3: Net-(Q3-Pad3) -> Net-(Q2-Pad3)
- U3 pad 4: Net-(R19-Pad2) -> Net-(R23-Pad2)
- U3 pad 8: VDD -> +5V
- U4 pad 1: Net-(R24-Pad2) -> Net-(R31-Pad2)
- U4 pad 2: Net-(Q4-Pad3) -> Net-(Q3-Pad3)
- U4 pad 3: Net-(Q4-Pad3) -> Net-(Q3-Pad3)
- U4 pad 4: Net-(R20-Pad2) -> Net-(R32-Pad2)
- U4 pad 8: VDD -> +5V
- U5 pad 1: Net-(R23-Pad1) -> Net-(R40-Pad2)
- U5 pad 2: Net-(R7-Pad1) -> Net-(Q4-Pad3)
- U5 pad 3: Net-(R36-Pad1) -> Net-(Q4-Pad3)
- U5 pad 4: Net-(R8-Pad1) -> Net-(R41-Pad2)
- U5 pad 5: Net-(R24-Pad1) -> GND
- U5 pad 6: GND -> Net-(J5-Pad1)
- U5 pad 7: GND -> Net-(J5-Pad2)
- U5 pad 8: GND -> +5V
Routing:
- removed copper zone on B.Cu, net GND
- removed copper zone on F.Cu, net GND
Other:
- board outline removed

Commit message: Transdutor
Signed-off-by: cuki2 <mauricio@krebs.com.br>
Routing:
- added copper zone on B.Cu, net GND
- added copper zone on F.Cu, net GND
Other:
- board outline added: 69.2 x 53.9 mm
Changed lines of the file:
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@@
   (general
     (links 140)
-    (no_connects 86)
-    (area 143.91053 46.4344 217.471601 105.4536)
+    (no_connects 81)
+    (area 148.080999 51.270999 217.431001 105.321001)
     (thickness 1.6)
-    (drawings 0)
+    (drawings 10)
     (tracks 0)
     (zones 0)
@@
     )
   )
+  (gr_line (start 214.756 105.246) (end 148.156 105.246) (angle 90) (layer Edge.Cuts) (width 0.15))
+  (gr_line (start 214.756 102.646) (end 214.756 105.246) (angle 90) (layer Edge.Cuts) (width 0.15))
+  (gr_line (start 217.356 100.046) (end 214.756 102.646) (angle 90) (layer Edge.Cuts) (width 0.15))
+  (gr_line (start 217.356 66.746) (end 217.356 100.046) (angle 90) (layer Edge.Cuts) (width 0.15))
+  (gr_line (start 214.856 64.246) (end 217.356 66.746) (angle 90) (layer Edge.Cuts) (width 0.15))
+  (gr_line (start 214.856 52.846) (end 214.856 64.246) (angle 90) (layer Edge.Cuts) (width 0.15))
+  (gr_line (start 214.756 52.746) (end 214.856 52.846) (angle 90) (layer Edge.Cuts) (width 0.15))
+  (gr_line (start 213.356 51.346) (end 214.756 52.746) (angle 90) (layer Edge.Cuts) (width 0.15))
+  (gr_line (start 148.156 51.346) (end 213.356 51.346) (angle 90) (layer Edge.Cuts) (width 0.15))
+  (gr_line (start 148.156 105.246) (end 148.156 51.346) (angle 90) (layer Edge.Cuts) (width 0.15))
+  (zone (net 1) (net_name GND) (layer F.Cu) (hatch edge 0.508)
+    (connect_pads (clearance 0.508))
+    (min_thickness 0.254)
+    (fill yes (arc_segments 16) (thermal_gap 0.508) (thermal_bridge_width 0.508))
+    (polygon
+      (pts
+        (xy 148.756 104.746) (xy 148.756 51.946) (xy 213.156 51.946) (xy 214.256 53.046) (xy 214.256 64.446)
+        (xy 216.756 67.046) (xy 216.756 99.746) (xy 216.756 99.846) (xy 214.256 102.346) (xy 214.256 104.746)
+      )
+    )
+  )
+  (zone (net 1) (net_name GND) (layer B.Cu) (hatch edge 0.508)
+    (connect_pads (clearance 0.508))
+    (min_thickness 0.254)
+    (fill yes (arc_segments 16) (thermal_gap 0.508) (thermal_bridge_width 0.508))
+    (polygon
+      (pts
+        (xy 148.756 104.746) (xy 148.756 51.946) (xy 213.156 51.946) (xy 214.256 53.046) (xy 214.256 64.446)
+        (xy 216.856 67.046) (xy 216.856 99.846) (xy 214.356 102.346) (xy 214.256 102.446) (xy 214.256 104.746)
+      )
+    )
+  )

Commit message: Signed-off-by: cuki2 <mauricio@krebs.com.br>
Parts:
- D1: value TX -> RX
- D2: value PWR -> TX
- D3: value RX -> PWR
- J1: value SL -> SL1; footprint w_pin_strip:pin_socket_3 -> w_pin_strip:pin_socket_2
- J2: value SL1 -> SL3
- J3: value SL2 -> SL4
- J4: value SL3 -> SL2
- J5: value SL4 -> SL; footprint w_pin_strip:pin_socket_2 -> w_pin_strip:pin_socket_3
- R1, R2: value 1k2 -> 10k
- R10: value 560R -> 360R
- R11, R26, R27: value 560R -> 10k
- R12: value 330R -> 10k
- R13: value 330R -> 120R
- R14, R33: value 10k -> 560R
- R15: value 10k -> 120R
- R16, R17: value 330R -> 560R
- R20, R24, R29, R3, R4: value 10k -> 360R
- R22, R23, R40, R6, R7: value 360R -> 10k
- R25, R9: value 120R -> 360R
- R31: value 360R -> 120R
- R32: value 360R -> 560R
- R37, R38, R42: value 10k -> 330R
- R41: value 360R -> 330R
- R43: value 120R -> 1k2
- R45: value 560R -> 1k2
- U2: value 4052 -> SP3481CP; footprint w_smd_dil:so-16 -> w_smd_dil:so-8
- U5: value SP3481CP -> 4052; footprint w_smd_dil:so-8 -> w_smd_dil:so-16
- moved J1 61.2 mm to (182.8, 115.3)
- moved J5 56.6 mm to (209.3, 59.4), turned to 180 degrees
- moved C1 46.9 mm to (182.8, 115.3)
- moved C2 46.9 mm to (182.8, 115.3)
- moved C3 46.9 mm to (182.8, 115.3)
- moved C4 46.9 mm to (182.8, 115.3)
- moved C5 46.9 mm to (182.8, 115.3)
- moved D3 46.9 mm to (182.8, 115.3)
- moved Q1 46.9 mm to (182.8, 115.3)
- moved Q2 46.9 mm to (182.8, 115.3)
- moved Q3 46.9 mm to (182.8, 115.3)
- moved Q4 46.9 mm to (182.8, 115.3)
- moved R1 46.9 mm to (182.8, 115.3)
- moved R10 46.9 mm to (182.8, 115.3)
- moved R11 46.9 mm to (182.8, 115.3)
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Connections:
- D1 pad 2: /TX -> Net-(D1-Pad2)
- D2 pad 1: +5V -> Net-(D2-Pad1)
- D2 pad 2: Net-(D2-Pad2) -> /TX
- D3 pad 1: Net-(D3-Pad1) -> +5V
- J1 pad 1: /TX -> Net-(J1-Pad1)
- J1 pad 2: /RX -> Net-(J1-Pad2)
- J5 pad 1: Net-(J5-Pad1) -> /RX
- J5 pad 2: Net-(J5-Pad2) -> /TX
- R1 pad 1: +5V -> Net-(Q1-Pad2)
- R1 pad 2: Net-(D1-Pad1) -> /RX1
- R10 pad 1: Net-(J2-Pad2) -> /TX3
- R10 pad 2: GND -> Net-(R10-Pad2)
- R11 pad 2: Net-(J2-Pad1) -> Net-(R11-Pad2)
- R12 pad 1: /ADR0 -> +5V
- R13 pad 1: /ADR1 -> Net-(J1-Pad1)
- R13 pad 2: Net-(R13-Pad2) -> Net-(J1-Pad2)
- R14 pad 1: GND -> Net-(J1-Pad2)
- R14 pad 2: Net-(R12-Pad2) -> GND
- R15 pad 1: GND -> Net-(J2-Pad1)
- R15 pad 2: Net-(R13-Pad2) -> Net-(J2-Pad2)
- R16 pad 1: /TX -> Net-(J2-Pad2)
- R16 pad 2: Net-(R16-Pad2) -> GND
- R17 pad 1: /RX -> +5V
- R17 pad 2: Net-(D3-Pad2) -> Net-(J1-Pad1)
- R18 pad 2: Net-(D3-Pad1) -> Net-(J2-Pad1)
- R19 pad 1: Net-(Q2-Pad2) -> Net-(Q3-Pad2)
- R19 pad 2: /RX2 -> /RX4
- R2 pad 1: GND -> Net-(Q2-Pad2)
- R2 pad 2: Net-(D2-Pad2) -> /RX3
- R20 pad 1: +5V -> /RX4
- R20 pad 2: Net-(Q2-Pad3) -> Net-(R20-Pad2)
- R21 pad 1: /TX2 -> /TX4
- R22 pad 1: /RX2 -> Net-(Q4-Pad2)
- R22 pad 2: Net-(R22-Pad2) -> /RX2
- R23 pad 1: /TX2 -> +5V
- R23 pad 2: Net-(R23-Pad2) -> Net-(Q3-Pad3)
- R24 pad 1: +5V -> /TX4
- R24 pad 2: Net-(R22-Pad2) -> Net-(R24-Pad2)
- R25 pad 1: Net-(J3-Pad1) -> /RX2
- R25 pad 2: Net-(J3-Pad2) -> Net-(R25-Pad2)
- R26 pad 1: Net-(J3-Pad2) -> +5V
- R26 pad 2: GND -> Net-(R20-Pad2)
- R27 pad 1: +5V -> /TX2
- R27 pad 2: Net-(J3-Pad1) -> +5V
- R28 pad 1: Net-(Q3-Pad2) -> +5V
- R28 pad 2: /RX3 -> Net-(Q4-Pad3)
- R29 pad 1: +5V -> /TX2
- R29 pad 2: Net-(Q3-Pad3) -> Net-(R29-Pad2)
- R3 pad 1: Net-(Q1-Pad2) -> /RX1
- R3 pad 2: /RX1 -> Net-(R11-Pad2)
- R30 pad 1: /TX3 -> +5V
- R30 pad 2: +5V -> Net-(R25-Pad2)
- R31 pad 1: /RX3 -> Net-(J3-Pad1)
- R31 pad 2: Net-(R31-Pad2) -> Net-(J3-Pad2)
- R32 pad 1: /TX3 -> Net-(J3-Pad2)
- R32 pad 2: Net-(R32-Pad2) -> GND
- R33 pad 2: Net-(R31-Pad2) -> Net-(J3-Pad1)
- R37 pad 1: Net-(Q4-Pad2) -> /ADR0
- R37 pad 2: /RX4 -> Net-(R37-Pad2)
- R38 pad 1: +5V -> /ADR1
- R38 pad 2: Net-(Q4-Pad3) -> Net-(R38-Pad2)
- R39 pad 1: /TX4 -> GND
- R39 pad 2: +5V -> Net-(R37-Pad2)
- R4 pad 1: +5V -> /RX3
- R4 pad 2: Net-(Q1-Pad3) -> Net-(R12-Pad2)
- R40 pad 1: /RX4 -> GND
- R40 pad 2: Net-(R40-Pad2) -> Net-(R38-Pad2)
- R41 pad 1: /TX4 -> /TX
- R42 pad 1: +5V -> /RX
- R42 pad 2: Net-(R40-Pad2) -> Net-(D1-Pad2)
- R43 pad 1: Net-(J5-Pad1) -> +5V
- R43 pad 2: Net-(J5-Pad2) -> Net-(D2-Pad1)
- R44 pad 1: Net-(J5-Pad2) -> +5V
- R44 pad 2: GND -> Net-(D1-Pad1)
- R45 pad 1: +5V -> GND
- R45 pad 2: Net-(J5-Pad1) -> Net-(D3-Pad2)
- R6 pad 1: /RX1 -> /TX3
- R6 pad 2: Net-(R6-Pad2) -> +5V
- R7 pad 1: /TX1 -> +5V
- R7 pad 2: Net-(R7-Pad2) -> Net-(Q1-Pad3)
- R8 pad 2: Net-(R6-Pad2) -> Net-(Q2-Pad3)
- R9 pad 1: Net-(J2-Pad1) -> /TX1
- R9 pad 2: Net-(J2-Pad2) -> Net-(R9-Pad2)
- U1 pad 1: Net-(R6-Pad2) -> Net-(R11-Pad2)
- U1 pad 4: Net-(R7-Pad2) -> Net-(R9-Pad2)
- U1 pad 6: Net-(J2-Pad1) -> Net-(J1-Pad1)
- U1 pad 7: Net-(J2-Pad2) -> Net-(J1-Pad2)
- U2 pad 1: /RX1 -> Net-(R12-Pad2)
- U2 pad 2: /RX3 -> Net-(Q2-Pad3)
- U2 pad 3: Net-(D3-Pad2) -> Net-(Q2-Pad3)
- U2 pad 4: /RX4 -> Net-(R10-Pad2)
- U2 pad 5: /RX2 -> GND
- U2 pad 6: GND -> Net-(J2-Pad1)
- U2 pad 7: GND -> Net-(J2-Pad2)
- U2 pad 8: GND -> +5V
- U3 pad 1: Net-(R22-Pad2) -> Net-(R20-Pad2)
- U3 pad 2: Net-(Q2-Pad3) -> Net-(Q3-Pad3)
- U3 pad 3: Net-(Q2-Pad3) -> Net-(Q3-Pad3)
- U3 pad 4: Net-(R23-Pad2) -> Net-(R24-Pad2)
- U4 pad 1: Net-(R31-Pad2) -> Net-(R25-Pad2)
- U4 pad 2: Net-(Q3-Pad3) -> Net-(Q4-Pad3)
- U4 pad 3: Net-(Q3-Pad3) -> Net-(Q4-Pad3)
- U4 pad 4: Net-(R32-Pad2) -> Net-(R29-Pad2)
- U5 pad 1: Net-(R40-Pad2) -> /RX1
- U5 pad 2: Net-(Q4-Pad3) -> /RX3
- U5 pad 3: Net-(Q4-Pad3) -> Net-(D1-Pad2)
- U5 pad 4: Net-(R41-Pad2) -> /RX4
- U5 pad 5: GND -> /RX2
- U5 pad 6: Net-(J5-Pad1) -> GND
- U5 pad 7: Net-(J5-Pad2) -> GND
- U5 pad 8: +5V -> GND
Routing:
- net Net-(D1-Pad2): track 0.00 -> 33.4 mm, vias 0 -> 2
- net Net-(R41-Pad2): track 0.00 -> 19.2 mm, vias 0 -> 2
- net /TX: track 0.00 -> 16.6 mm
- net /RX: track 0.00 -> 9.43 mm
- net Net-(D2-Pad1): track 0.00 -> 2.82 mm
- net Net-(D1-Pad1): track 0.00 -> 2.82 mm
- net +5V: track 0.00 -> 2.29 mm
