File: MultiplexadorSerial/sch/MuxDemux.sch (KiCad schematic (older format))
At the start: 10 parts, among them U2 4052

Commit message: Transdutor
Signed-off-by: cuki2 <mauricio@krebs.com.br>
Parts:
- renumbered C2 to C1, R12 to R3, R13 to R4, R14 to R5, R15 to R6, R16 to R7, R17 to R8, R18 to R9, U2 to U1
Changed lines of the file:
@@
 $Descr A4 11693 8268
 encoding utf-8
-Sheet 3 6
+Sheet 3 3
 Title "Multiplexador serial rs485"
-Date "2017-11-27"
+Date "2017-11-28"
 Rev "0"
 Comp "Krebsfer Industrial LTDA."
@@
 $EndDescr
 $Comp
-L 4052 U2
+L 4052 U1
 U 1 1 5A1FBFC5
 P 5950 3850
-F 0 "U2" H 6050 3850 50  0000 C CNN
+F 0 "U1" H 6050 3850 50  0000 C CNN
 F 1 "4052" H 6050 3650 50  0000 C CNN
 F 2 "w_smd_dil:so-16" H 5950 3850 60  0001 C CNN
@@
 $EndComp
 $Comp
-L C C2
+L C C1
 U 1 1 5A1FBFCC
 P 4500 3600
-F 0 "C2" H 4525 3700 50  0000 L CNN
+F 0 "C1" H 4525 3700 50  0000 L CNN
 F 1 "100nF" H 4525 3500 50  0000 L CNN
 F 2 "w_smd_cap:c_0805" H 4538 3450 50  0001 C CNN
@@
 $EndComp
 $Comp
-L GND #PWR017
+L GND #PWR08
 U 1 1 5A1FBFD3
 P 4500 3850
-F 0 "#PWR017" H 4500 3600 50  0001 C CNN
+F 0 "#PWR08" H 4500 3600 50  0001 C CNN
 F 1 "GND" H 4500 3700 50  0000 C CNN
 F 2 "" H 4500 3850 50  0001 C CNN
@@
 $EndComp
 $Comp
-L GND #PWR018
+L GND #PWR09
 U 1 1 5A1FBFD9
 P 5950 4600
-F 0 "#PWR018" H 5950 4350 50  0001 C CNN
+F 0 "#PWR09" H 5950 4350 50  0001 C CNN
 F 1 "GND" H 5950 4450 50  0000 C CNN
 F 2 "" H 5950 4600 50  0001 C CNN
@@
 $EndComp
 $Comp
-L R R16
+L R R7
 U 1 1 5A1FBFDF
 P 6850 3250
-F 0 "R16" V 6930 3250 50  0000 C CNN
+F 0 "R7" V 6930 3250 50  0000 C CNN
 F 1 "330R" V 6850 3250 50  0000 C CNN
 F 2 "w_smd_resistors:r_0805" V 6780 3250 50  0001 C CNN
@@
 $EndComp
 $Comp
-L R R17
+L R R8
 U 1 1 5A1FBFE6
 P 7000 3650
-F 0 "R17" V 7080 3650 50  0000 C CNN
+F 0 "R8" V 7080 3650 50  0000 C CNN
 F 1 "330R" V 7000 3650 50  0000 C CNN
 F 2 "w_smd_resistors:r_0805" V 6930 3650 50  0001 C CNN
@@
 $EndComp
 $Comp
-L R R13
+L R R4
 U 1 1 5A1FBFED
 P 4800 4550
-F 0 "R13" V 4880 4550 50  0000 C CNN
+F 0 "R4" V 4880 4550 50  0000 C CNN
 F 1 "330R" V 4800 4550 50  0000 C CNN
 F 2 "w_smd_resistors:r_0805" V 4730 4550 50  0001 C CNN
@@
 $EndComp
 $Comp
-L R R12
+L R R3
 U 1 1 5A1FBFF4
 P 4800 4350
-F 0 "R12" V 4880 4350 50  0000 C CNN
+F 0 "R3" V 4880 4350 50  0000 C CNN
 F 1 "330R" V 4800 4350 50  0000 C CNN
 F 2 "w_smd_resistors:r_0805" V 4730 4350 50  0001 C CNN
@@
 $EndComp
 $Comp
-L R R18
+L R R9
 U 1 1 5A1FC002
 P 7400 3900
-F 0 "R18" V 7480 3900 50  0000 C CNN
+F 0 "R9" V 7480 3900 50  0000 C CNN
 F 1 "560R" V 7400 3900 50  0000 C CNN
 F 2 "w_smd_resistors:r_0805" V 7330 3900 50  0001 C CNN
@@
 $EndComp
 $Comp
-L GND #PWR019
+L GND #PWR010
 U 1 1 5A1FC009
 P 5050 4100
-F 0 "#PWR019" H 5050 3850 50  0001 C CNN
+F 0 "#PWR010" H 5050 3850 50  0001 C CNN
 F 1 "GND" H 5050 3950 50  0000 C CNN
 F 2 "" H 5050 4100 50  0001 C CNN
@@
 $EndComp
 $Comp
-L R R15
+L R R6
 U 1 1 5A1FC00F
 P 5300 4850
-F 0 "R15" V 5380 4850 50  0000 C CNN
+F 0 "R6" V 5380 4850 50  0000 C CNN
 F 1 "10k" V 5300 4850 50  0000 C CNN
 F 2 "w_smd_resistors:r_0805" V 5230 4850 50  0001 C CNN
@@
 $EndComp
 $Comp
-L +5V #PWR020
+L +5V #PWR011
 U 1 1 5A1FC016
 P 5950 3050
-F 0 "#PWR020" H 5950 2900 50  0001 C CNN
+F 0 "#PWR011" H 5950 2900 50  0001 C CNN
 F 1 "+5V" H 5950 3190 50  0000 C CNN
 F 2 "" H 5950 3050 50  0001 C CNN
@@
 $EndComp
 $Comp
-L +5V #PWR021
+L +5V #PWR012
 U 1 1 5A1FC01C
 P 4500 3400
-F 0 "#PWR021" H 4500 3250 50  0001 C CNN
+F 0 "#PWR012" H 4500 3250 50  0001 C CNN
 F 1 "+5V" H 4500 3540 50  0000 C CNN
 F 2 "" H 4500 3400 50  0001 C CNN
@@
 $EndComp
 $Comp
-L GND #PWR022
+L GND #PWR013
 U 1 1 5A1FC022
 P 6750 4400
-F 0 "#PWR022" H 6750 4150 50  0001 C CNN
+F 0 "#PWR013" H 6750 4150 50  0001 C CNN
 F 1 "GND" H 6750 4250 50  0000 C CNN
 F 2 "" H 6750 4400 50  0001 C CNN
@@
 $EndComp
 $Comp
-L +5V #PWR023
+L +5V #PWR014
 U 1 1 5A1FC02A
 P 7650 3850
-F 0 "#PWR023" H 7650 3700 50  0001 C CNN
+F 0 "#PWR014" H 7650 3700 50  0001 C CNN
 F 1 "+5V" H 7650 3990 50  0000 C CNN
 F 2 "" H 7650 3850 50  0001 C CNN
@@
 $EndComp
 $Comp
-L R R14
+L R R5
 U 1 1 5A1FC044
 P 5050 4850
-F 0 "R14" V 5130 4850 50  0000 C CNN
+F 0 "R5" V 5130 4850 50  0000 C CNN
 F 1 "10k" V 5050 4850 50  0000 C CNN
 F 2 "w_smd_resistors:r_0805" V 4980 4850 50  0001 C CNN
@@
 $EndComp
 $Comp
-L GND #PWR024
+L GND #PWR015
 U 1 1 5A1FC04B
 P 5300 5050
-F 0 "#PWR024" H 5300 4800 50  0001 C CNN
+F 0 "#PWR015" H 5300 4800 50  0001 C CNN
 F 1 "GND" H 5300 4900 50  0000 C CNN
 F 2 "" H 5300 5050 50  0001 C CNN
@@
 $EndComp
 $Comp
-L GND #PWR025
+L GND #PWR016
 U 1 1 5A1FC051
 P 5050 5050
-F 0 "#PWR025" H 5050 4800 50  0001 C CNN
+F 0 "#PWR016" H 5050 4800 50  0001 C CNN
 F 1 "GND" H 5050 4900 50  0000 C CNN
 F 2 "" H 5050 5050 50  0001 C CNN
@@
 	6700 4350 6650 4350
 Wire Wire Line
-	6650 3650 6750 3650
-Wire Wire Line
-	6750 3650 6850 3650
+	6650 3650 6850 3650
 Wire Wire Line
 	7100 3250 7000 3250
@@
 	7600 3900 7550 3900
 Wire Wire Line
-	4950 4350 5050 4350
-Wire Wire Line
-	5050 4350 5250 4350
+	4950 4350 5250 4350
 Wire Wire Line
 	4950 4550 5150 4550
 Wire Wire Line
-	5150 4450 5150 4550
-Wire Wire Line
-	5150 4550 5150 4600
+	5150 4450 5150 4600
 Wire Wire Line
 	5150 4450 5250 4450
