File: MultiplexadorSerial/sch/Transdutor.sch (KiCad schematic (older format))
At the start: 13 parts, among them J2 SL1, Q1 Q_NPN_CBE, U1 SP3481CP

Commit message: Transdutor
Signed-off-by: cuki2 <mauricio@krebs.com.br>
Parts:
- added C2, C3, C5: 100nF, w_smd_cap:c_0805, symbol C
- added J2: SL4, w_pin_strip:pin_socket_2, symbol CONN_01X02
- added J3: SL1, w_pin_strip:pin_socket_2, symbol CONN_01X02
- added J5: SL3, w_pin_strip:pin_socket_2, symbol CONN_01X02
- added Q1, Q2, Q4: Q_NPN_CBE, w_smd_trans:sot23, symbol Q_NPN_EBC
- added R10, R12, R13, R15, R16, R18, R19, R21, R37, R39, R40, R42: 10k, w_smd_resistors:r_0805, symbol R
- added R11, R14, R17, R20, R38, R41: 360R, w_smd_resistors:r_0805, symbol R
- added R22, R24, R43: 120R, w_smd_resistors:r_0805, symbol R
- added R23, R25, R26, R27, R44, R45: 560R, w_smd_resistors:r_0805, symbol R
- added U2, U3, U5: SP3481CP, w_smd_dil:so-8, symbol SP3481CP
- J4: renamed from J2; value SL1 -> SL2
- renumbered C1 to C4, Q1 to Q3, R3 to R28, R6 to R29, R5 to R30, R4 to R31, R7 to R32, R8 to R33, R9 to R34, R10 to R35, R11 to R36, U1 to U4
Connections:
- net +5V: now also C2.1, C3.1, C5.1, R13.2, R15.1, R16.2, R18.1, R19.1, R21.1, R26.1, R27.1, R39.2, R40.1, R42.1, R45.1, U2.8 (VCC), U3.8 (VCC), U5.8 (VCC)
- net GND: now also C2.2, C3.2, C5.2, Q1.1 (E), Q2.1 (E), Q4.1 (E), R23.2, R25.2, R44.2, U2.5 (GND), U3.5 (GND), U5.5 (GND)
- net RX renamed RX2
- net TX renamed TX2
- new net: R14.2, R21.2, U3.1 (RO)
- new net: Q2.3 (C), R18.2, U3.2 (~RE~), U3.3 (DE)
- new net: R20.2, U3.4 (DI)
- new net: J3.1 (P1), R24.1, R27.2, U3.6 (A)
- new net: J3.2 (P2), R24.2, R25.1, U3.7 (B)
- new net: Q2.2 (B), R12.1
- new net: R11.2, R19.2, U2.1 (RO)
- new net: Q1.3 (C), R15.2, U2.2 (~RE~), U2.3 (DE)
- new net: R17.2, U2.4 (DI)
- new net: J2.1 (P1), R22.1, R26.2, U2.6 (A)
- new net: J2.2 (P2), R22.2, R23.1, U2.7 (B)
- new net: Q1.2 (B), R10.1
- new net: R38.2, R42.2, U5.1 (RO)
- new net: Q4.3 (C), R40.2, U5.2 (~RE~), U5.3 (DE)
- new net: R41.2, U5.4 (DI)
- new net: J5.1 (P1), R43.1, R45.2, U5.6 (A)
- new net: J5.2 (P2), R43.2, R44.1, U5.7 (B)
- new net: Q4.2 (B), R37.1
- new net RX1: R12.2, R14.1
- new net RX3: R37.2, R38.1
- new net RX4: R10.2, R11.1
- new net TX1: R16.1, R20.1
- new net TX3: R39.1, R41.1
- new net TX4: R13.1, R17.1
