File: MultiplexadorSerial/sch/MultiplexadorSerial.sch (KiCad schematic (older format))
At the start: 6 parts, among them J1 SL

Commit message: Transdutor
Signed-off-by: cuki2 <mauricio@krebs.com.br>
Changed lines of the file:
@@
 $Descr A4 11693 8268
 encoding utf-8
-Sheet 1 6
+Sheet 1 3
 Title "Multiplexador serial rs485"
-Date "2017-11-27"
+Date "2017-11-28"
 Rev "0"
 Comp "Krebsfer Industrial LTDA."
@@
 	-1   0    0    -1
 $EndComp
-$Sheet
-S 3150 2750 550  200
-U 5A1D0C3D
-F0 "Transdutor" 60
-F1 "Transdutor.sch" 60
-F2 "TX" I R 3700 2800 60
-F3 "RX" O R 3700 2900 60
-$EndSheet
 $Comp
 L GND #PWR03
@@
 	5500 3550 5800 3550
 Wire Wire Line
-	4850 3150 4600 3150
-Wire Wire Line
-	4850 3250 4600 3250
-Wire Wire Line
-	4850 3350 4600 3350
-Wire Wire Line
-	4850 3450 4600 3450
-Wire Wire Line
-	4850 3550 4600 3550
-Wire Wire Line
-	4850 3650 4600 3650
-Wire Wire Line
-	4850 3750 4600 3750
-Wire Wire Line
-	4850 3850 4600 3850
-Text Label 4600 3150 0    60   ~ 0
-TX1
-Text Label 4600 3350 0    60   ~ 0
-TX2
-Text Label 4600 3550 0    60   ~ 0
-TX3
-Text Label 4600 3750 0    60   ~ 0
-TX4
-Text Label 4600 3250 0    60   ~ 0
-RX1
-Text Label 4600 3450 0    60   ~ 0
-RX2
-Text Label 4600 3650 0    60   ~ 0
-RX3
-Text Label 4600 3850 0    60   ~ 0
-RX4
-Wire Wire Line
 	8400 4500 8200 4500
 Wire Wire Line
@@
 Text Label 5800 3550 2    60   ~ 0
 ADR1
-Text Label 4150 2800 2    60   ~ 0
-TX1
-Wire Wire Line
-	4150 2800 3700 2800
-Text Label 4150 2900 2    60   ~ 0
-RX1
-Wire Wire Line
-	4150 2900 3700 2900
-$Sheet
-S 3150 3150 550  200
-U 5A211D6C
-F0 "Transdutor" 60
-F1 "Transdutor.sch" 60
-F2 "TX" I R 3700 3200 60
-F3 "RX" O R 3700 3300 60
-$EndSheet
-Wire Wire Line
-	4150 3200 3700 3200
-Wire Wire Line
-	4150 3300 3700 3300
-$Sheet
-S 3150 3600 550  200
-U 5A212104
-F0 "Transdutor" 60
-F1 "Transdutor.sch" 60
-F2 "TX" I R 3700 3650 60
-F3 "RX" O R 3700 3750 60
-$EndSheet
-Wire Wire Line
-	4150 3650 3700 3650
-Wire Wire Line
-	4150 3750 3700 3750
-$Sheet
-S 3150 4000 550  200
-U 5A21210C
-F0 "Transdutor" 60
-F1 "Transdutor.sch" 60
-F2 "TX" I R 3700 4050 60
-F3 "RX" O R 3700 4150 60
-$EndSheet
-Wire Wire Line
-	4150 4050 3700 4050
-Wire Wire Line
-	4150 4150 3700 4150
-Text Label 4150 3200 2    60   ~ 0
-TX2
-Text Label 4150 3300 2    60   ~ 0
-RX2
-Text Label 4150 3650 2    60   ~ 0
-TX3
-Text Label 4150 3750 2    60   ~ 0
-RX3
-Text Label 4150 4050 2    60   ~ 0
-TX4
-Text Label 4150 4150 2    60   ~ 0
-RX4
 $Comp
 L GND #PWR07
@@
 Wire Wire Line
 	8250 4700 8200 4700
+$Sheet
+S 3850 3100 550  800
+U 5A1D0C3D
+F0 "Transdutor" 60
+F1 "Transdutor.sch" 60
+F2 "TX2" I R 4400 3350 60
+F3 "RX2" O R 4400 3450 60
+F4 "TX1" I R 4400 3150 60
+F5 "RX1" O R 4400 3250 60
+F6 "TX4" I R 4400 3750 60
+F7 "RX4" O R 4400 3850 60
+F8 "TX3" I R 4400 3550 60
+F9 "RX3" O R 4400 3650 60
+$EndSheet
+Wire Wire Line
+	4850 3150 4400 3150
+Wire Wire Line
+	4850 3250 4400 3250
+Wire Wire Line
+	4850 3350 4400 3350
+Wire Wire Line
+	4850 3450 4400 3450
+Wire Wire Line
+	4850 3550 4400 3550
+Wire Wire Line
+	4850 3650 4400 3650
+Wire Wire Line
+	4850 3750 4400 3750
+Wire Wire Line
+	4850 3850 4400 3850
 $EndSCHEMATC

Commit message: Signed-off-by: cuki2 <mauricio@krebs.com.br>
Parts:
- added C1, C2, C3, C4, C5: 100nF, w_smd_cap:c_0805, symbol C
- added D1: RX, w_smd_leds:Led_0805, symbol M_LED
- added J1: SL1, w_pin_strip:pin_socket_2, symbol CONN_01X02
- added J2: SL3, w_pin_strip:pin_socket_2, symbol CONN_01X02
- added J3: SL4, w_pin_strip:pin_socket_2, symbol CONN_01X02
- added J4: SL2, w_pin_strip:pin_socket_2, symbol CONN_01X02
- added Q1, Q2, Q3, Q4: Q_NPN_CBE, w_smd_trans:sot23, symbol Q_NPN_EBC
- added R1, R11, R12, R19, R2, R21, R22, R23, R26, R27, R28, R30, R39, R40, R5, R6, R7, R8: 10k, w_smd_resistors:r_0805, symbol R
- added R10, R20, R24, R25, R29, R3, R4, R9: 360R, w_smd_resistors:r_0805, symbol R
- added R13, R15, R31, R34: 120R, w_smd_resistors:r_0805, symbol R
- added R14, R16, R17, R18, R32, R33, R35, R36, R44: 560R, w_smd_resistors:r_0805, symbol R
- added R37, R38, R41, R42: 330R, w_smd_resistors:r_0805, symbol R
- added U1, U2, U3, U4: SP3481CP, w_smd_dil:so-8, symbol SP3481CP
- added U5: 4052, w_smd_dil:so-16, symbol 4052
- renumbered D1 to D2, D2 to D3, J1 to J5, R1 to R43, R2 to R45
Connections:
- net +5V: now also C1.1, C2.1, C3.1, C4.1, C5.1, R11.1, R12.1, R17.1, R18.1, R21.2, R23.1, R26.1, R27.2, R28.1, R30.1, R33.1, R36.1, R44.1, R5.2, R6.2, R7.1, R8.1, U1.8 (VCC), U2.8 (VCC), U3.8 (VCC), U4.8 (VCC), U5.16 (VDD)
- net ADR0: now also R37.1
- net ADR1: now also R38.1
- net GND: now also C1.2, C2.2, C3.2, C4.2, C5.2, Q1.1 (E), Q2.1 (E), Q3.1 (E), Q4.1 (E), R14.2, R16.2, R32.2, R35.2, R39.1, R40.1, U1.5 (GND), U2.5 (GND), U3.5 (GND), U4.5 (GND), U5.6 (Inh), U5.7 (VEE), U5.8 (VSS)
- net RX: now also J5.1 (P1), R42.1; no longer J5.2 (P2)
- net TX: now also J5.2 (P2), R41.1; no longer J5.1 (P1)
- new net: R25.2, R30.2, U4.1 (RO)
- new net: Q4.3 (C), R28.2, U4.2 (~RE~), U4.3 (DE)
- new net: R29.2, U4.4 (DI)
- new net: J4.1 (P1), R34.1, R36.2, U4.6 (A)
- new net: J4.2 (P2), R34.2, R35.1, U4.7 (B)
- new net: Q4.2 (B), R22.1
- new net: R11.2, R3.2, U1.1 (RO)
- new net: Q1.3 (C), R7.2, U1.2 (~RE~), U1.3 (DE)
- new net: R9.2, U1.4 (DI)
- new net: J1.1 (P1), R13.1, R17.2, U1.6 (A)
- new net: J1.2 (P2), R13.2, R14.1, U1.7 (B)
- new net: Q1.2 (B), R1.1
- new net: R20.2, R26.2, U3.1 (RO)
- new net: Q3.3 (C), R23.2, U3.2 (~RE~), U3.3 (DE)
- new net: R24.2, U3.4 (DI)
- new net: J3.1 (P1), R31.1, R33.2, U3.6 (A)
- new net: J3.2 (P2), R31.2, R32.1, U3.7 (B)
- new net: Q3.2 (B), R19.1
- new net: R12.2, R4.2, U2.1 (RO)
- new net: Q2.3 (C), R8.2, U2.2 (~RE~), U2.3 (DE)
- new net: R10.2, U2.4 (DI)
- new net: J2.1 (P1), R15.1, R18.2, U2.6 (A)
- new net: J2.2 (P2), R15.2, R16.1, U2.7 (B)
- new net: Q2.2 (B), R2.1
- new net: R37.2, R39.2, U5.10 (A)
- new net: R41.2, U5.13 (X)
- new net: D1.2 (K), R42.2, U5.3 (Y)
- new net: R38.2, R40.2, U5.9 (B)
- new net: D1.1 (A), R44.2
- new net RX1: R1.2, R3.1, U5.1 (Y0)
- new net RX2: R22.2, R25.1, U5.5 (Y1)
- new net RX3: R2.2, R4.1, U5.2 (Y2)
- new net RX4: R19.2, R20.1, U5.4 (Y3)
- new net TX1: R5.1, R9.1, U5.12 (X0)
- new net TX2: R27.1, R29.1, U5.14 (X1)
- new net TX3: R10.1, R6.1, U5.15 (X2)
- new net TX4: R21.1, R24.1, U5.11 (X3)
Other:
- moved on the sheet: D2, D3, J5, R43, R45, SHIELD1
