File: ReleModbus/sch/ReleModbus.sch (KiCad schematic (older format))
At the start: 47 parts, among them J1 PWR, J2 ICSP, J3 I2C, J4 DB9_FEMALE, J5 COMUM, J6 N_ABERTO, J7 N_FECHADO, Q1 BC817, Q2 BC817, U1 ATMEGA328P-AU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

Commit message: Signed-off-by: cuki2 <mauricio@krebs.com.br>
Parts:
- D1, D2, D3: symbol D_ALT -> D_ALT-RESCUE-ReleModbus
Changed lines of the file:
@@
 EESchema Schematic File Version 2
+LIBS:ReleModbus-rescue
 LIBS:power
 LIBS:device
@@
 encoding utf-8
 Sheet 1 1
-Title ""
-Date ""
-Rev ""
+Title "ReleModbus"
+Date "2017-12-06"
+Rev "0"
 Comp ""
 Comment1 ""
-Comment2 ""
-Comment3 ""
-Comment4 ""
+Comment2 "mauriciocukier@gmail.com"
+Comment3 "Engenheiro Eletrico"
+Comment4 "Mauricio Cukier"
 $EndDescr
 $Comp
-L D_ALT D1
+L D_ALT-RESCUE-ReleModbus D1
 U 1 1 5A27DCAF
 P 2050 950
@@
 SCL
 $Comp
-L D_ALT D2
+L D_ALT-RESCUE-ReleModbus D2
 U 1 1 5A2920A2
 P 6700 1350
@@
 	6150 2700 6150 2600
 $Comp
-L D_ALT D3
+L D_ALT-RESCUE-ReleModbus D3
 U 1 1 5A294797
 P 6700 3000

Commit message: Signed-off-by: cuki2 <mauricio@krebs.com.br>
Parts:
- C9: value 470uF 10V -> 470uF 25V; footprint w_capacitors:CP_8x7mm -> w_capacitors:CP_6.3x11mm
- D6: value LED -> PWR
Other:
- moved on the sheet: C1, C2, C3, C4, D4, D5, D6, J2, J3, J4, R1, R10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

Commit message: Signed-off-by: cuki2 <mauricio@krebs.com.br>
Parts:
- removed U1: ATMEGA328P-AU, w_smd_lqfp:lqfp32, symbol ATMEGA328P-AU
- added U1: ATMEGA328P-PU, w_pth_circuits:dil_28-300, symbol ATMEGA328P-PU
Connections:
- net +5V: now also U1.20 (AVCC), U1.7 (VCC)
- net GND: now also U1.22 (GND), U1.8 (GND)
- net MISO: now also U1.18 ((PCINT4/MISO)PB4)
- net MOSI: now also U1.17 ((PCINT3/OC2A/MOSI)PB3)
- net RST: now also U1.1 ((PCINT14/~RESET~)PC6)
- net RX_TTL: now also U1.2 ((PCINT16/RXD)PD0)
- net R_EN: now also U1.25 ((PCINT10/ADC2)PC2)
- net SCK: now also U1.19 ((PCINT5/SCK)PB5)
- net SCL: now also U1.28 ((PCINT13/SCL/ADC5)PC5)
- net SDA: now also U1.27 ((PCINT12/SDA/ADC4)PC4)
- net TX_TTL: now also U1.3 ((PCINT17/TXD)PD1)
- net XTAL1: now also U1.9 ((PCINT6/XTAL1/TOSC1)PB6)
- net XTAL2: now also U1.10 ((PCINT7/XTAL2/TOSC2)PB7)
- no-connect marks 19 -> 18
