File: ReleModbus/sch/ReleModbus.kicad_pcb (KiCad board)
At the start: 2 copper layers, 66 x 71 mm, 47 parts, among them J1 PWR, J2 ICSP, J3 I2C, J4 DB9_FEMALE, J5 COMUM, J6 N_ABERTO, J7 N_FECHADO, Q1 BC817, Q2 BC817, U1 ATMEGA328P-AU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

Commit message: Signed-off-by: cuki2 <mauricio@krebs.com.br>
Parts:
- added hole_3mm: VAL**, w_details:hole_3mm, F.Cu at (78.0, 18.0)
- added hole_3mm: VAL**, w_details:hole_3mm, F.Cu at (28.0, 18.0)
- added hole_3mm: VAL**, w_details:hole_3mm, F.Cu at (28.0, 89.0)
- added hole_3mm: VAL**, w_details:hole_3mm, F.Cu at (78.0, 89.0)
- C7: moved to F.Cu
- moved C7 21.8 mm to (46.4, 41.8), turned to 90 degrees
- moved RV1 16.2 mm to (23.2, 23.7)
- moved J1 12.8 mm to (36.6, 20.1), turned to 180 degrees
- moved J7 10.7 mm to (36.8, 87.0)
- moved C6 10.5 mm to (36.2, 33.0)
- moved J6 10.2 mm to (47.5, 87.0)
- moved J5 9.72 mm to (58.2, 87.0)
- moved U2 5.14 mm to (50.0, 29.7)
- moved D1 3.33 mm to (30.1, 27.9), turned to 0 degrees
- moved R10 0.08 mm to (62.0, 30.3)
Routing:
- net /NF2: track 73.3 -> 48.4 mm
- net Net-(C6-Pad1): track 38.1 -> 24.8 mm
- net /NF1: track 82.7 -> 71.6 mm
- net /NA2: track 44.6 -> 34.1 mm
- net /C1: track 71.2 -> 63.6 mm
- net /NA1: track 56.2 -> 52.3 mm
- net Net-(D1-Pad1): track 22.1 -> 25.5 mm
- net /C2: track 18.7 -> 21.9 mm
- net Net-(D3-Pad1): track 17.8 -> 20.5 mm
- net +5V: track 183.8 -> 186.0 mm
Other:
- board size 66 x 71 mm -> 66 x 77 mm
- net class PWR: clearance 0.1 -> 0.2

Commit message: Signed-off-by: cuki2 <mauricio@krebs.com.br>
Parts:
- C9: value 470uF 10V -> 470uF 25V; footprint w_capacitors:CP_8x7mm -> w_capacitors:CP_6.3x11mm
- U1: value ATMEGA328P-AU -> ATMEGA328P-PU; footprint w_smd_lqfp:lqfp32 -> w_pth_circuits:dil_28-300
- moved C9 21.6 mm to (58.7, 39.6), turned to 180 degrees
- moved J3 21.4 mm to (24.9, 85.3), turned to 180 degrees
- moved C1 20.8 mm to (42.7, 62.5), turned to 180 degrees
- moved C11 20.4 mm to (27.7, 55.4), turned to 270 degrees
- moved C8 11.8 mm to (53.6, 42.2)
- moved J2 11.7 mm to (24.9, 79.2), turned to 90 degrees
- moved R8 10.9 mm to (44.7, 49.3), turned to 0 degrees
- moved R9 10.8 mm to (26.9, 40.4)
- moved R2 9.24 mm to (42.7, 42.2), turned to 0 degrees
- moved R7 9.02 mm to (44.7, 51.6), turned to 0 degrees
- moved C3 8.03 mm to (45.7, 59.2), turned to 0 degrees
- moved R1 6.02 mm to (42.7, 44.7), turned to 0 degrees
- moved C10 4.44 mm to (59.9, 59.4)
- moved C12 4.44 mm to (59.9, 54.1)
- moved C14 4.44 mm to (59.9, 48.8), turned to 90 degrees
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Connections:
- U1 pad 1: Net-(U1-Pad1) -> /RST
- U1 pad 10: Net-(U1-Pad10) -> /XTAL2
- U1 pad 15: /MOSI -> Net-(U1-Pad15)
- U1 pad 16: /MISO -> Net-(U1-Pad16)
- U1 pad 17: /SCK -> /MOSI
- U1 pad 18: +5V -> /MISO
- U1 pad 19: Net-(U1-Pad19) -> /SCK
- U1 pad 2: Net-(U1-Pad2) -> /RX_TTL
- U1 pad 21: GND -> Net-(U1-Pad21)
- U1 pad 22: Net-(U1-Pad22) -> GND
- U1 pad 3: GND -> /TX_TTL
- U1 pad 4: +5V -> Net-(U1-Pad4)
- U1 pad 5: GND -> Net-(U1-Pad5)
- U1 pad 6: +5V -> Net-(U1-Pad6)
- U1 pad 7: /XTAL1 -> +5V
- U1 pad 8: /XTAL2 -> GND
- U1 pad 9: Net-(U1-Pad9) -> /XTAL1
Routing:
- net GND: track 59.3 -> 244.3 mm, vias 5 -> 0
- net /SCL: track 23.6 -> 60.6 mm
- net Net-(R8-Pad1): track 33.0 -> 4.35 mm, vias 2 -> 0
- net /SDA: track 25.6 -> 52.2 mm
- net Net-(R7-Pad1): track 28.8 -> 3.93 mm, vias 2 -> 0
- net /RX_TTL: track 3.74 -> 23.1 mm
- net /MISO: track 12.4 -> 29.0 mm
- net /R_EN: track 27.8 -> 44.2 mm, vias 2 -> 1
- net /C1: track 63.6 -> 47.3 mm
- net /MOSI: track 9.88 -> 23.8 mm, vias 1 -> 0
- net /SCK: track 10.4 -> 24.1 mm
- net +5V: track 186.0 -> 199.6 mm, vias 4 -> 1
- net /C2: track 21.9 -> 10.8 mm
- net /TX_TTL: track 4.12 -> 13.6 mm
- net /RST: track 32.8 -> 42.0 mm, vias 2 -> 0
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- removed copper zone on B.Cu, net GND
- removed copper zone on F.Cu, net GND
Other:
- net class Default: trace_width 0.25 -> 0.3; via_dia 1 -> 1.5; via_drill 0.8 -> 1
- net class PWR: via_dia 1 -> 1.5; via_drill 0.8 -> 1

Commit message: Gerber Rele Modbus R0
Signed-off-by: maurice <mauricio@krebs.com.br>
Parts:
- D2, D3, Q1, Q2, R3, R4, R5, R6: moved to B.Cu
- moved R6 17.7 mm to (71.9, 80.3)
- moved R4 13.7 mm to (61.2, 79.0)
- moved D2 12.8 mm to (68.8, 61.0)
- moved Q2 12.7 mm to (63.2, 82.5), turned to 0 degrees
- moved Q1 12.5 mm to (63.8, 68.3), turned to 90 degrees
- moved R3 12.1 mm to (59.4, 69.3)
- moved D3 10.6 mm to (69.1, 79.8)
- moved R5 10.5 mm to (64.3, 64.8), turned to 0 degrees
Routing:
- net GND: track 244.3 -> 199.2 mm
- net +5V: track 199.6 -> 217.8 mm
- net Net-(D3-Pad1): track 20.0 -> 11.0 mm
- net Net-(D2-Pad1): track 17.7 -> 12.0 mm
- net /R_EN: track 44.2 -> 45.0 mm, vias 1 -> 2
- added copper zone on B.Cu, net GND
- added copper zone on F.Cu, net GND
