File: Trena/sch/Trena.kicad_pcb (KiCad board)
At the start: 2 copper layers, 70.7 x 70.7 mm, 49 parts, among them J1 RJ45, J2 ICSP, J4 IN, J5 OUT, Q1 PN2222A, Q2 BC817-40, Q3 BC817-40, U1 ATMEGA328P-AU, U2 LM1117-5.0, U3 SP3485CN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

Commit message: Trilhas Trena Serial
Signed-off-by: cuki2 <mauricio@krebs.com.br>
Parts:
- moved J2 17.8 mm to (46.7, 81.8), turned to 180 degrees
- moved F1 15.4 mm to (38.6, 19.8), turned to 270 degrees
- moved R16 8.73 mm to (81.5, 54.4), turned to 90 degrees
- moved R15 8.13 mm to (80.3, 63.0), turned to 90 degrees
- moved D7 7.18 mm to (49.8, 33.5)
- moved R20 5.18 mm to (56.9, 33.5)
- moved D4 3.05 mm to (73.2, 64.5)
- moved D5 3.05 mm to (76.2, 64.5)
- moved R7 3.05 mm to (76.2, 68.6)
- moved R9 3.05 mm to (73.2, 68.6)
- moved D1 1.61 mm to (38.6, 26.4)
- moved C8 0.99 mm to (25.4, 28.4)
- moved U2 0.97 mm to (31.5, 26.4)
- moved C7 0.85 mm to (33.5, 21.3)
- moved C4 0.51 mm to (46.7, 66.0)
Connections:
- U1 pad 7: /XTAL1 -> /XTAL2
- U1 pad 8: /XTAL2 -> /XTAL1
Routing:
- net +5V: track 0.00 -> 254.9 mm, vias 0 -> 4
- net GND: track 0.00 -> 159.2 mm, vias 0 -> 8
- net /LED1: track 0.00 -> 85.0 mm, vias 0 -> 1
- net /INT2: track 0.00 -> 73.1 mm, vias 0 -> 2
- net /A: track 0.00 -> 72.6 mm, vias 0 -> 3
- net /B: track 0.00 -> 71.9 mm, vias 0 -> 1
- net /LED2: track 0.00 -> 61.0 mm, vias 0 -> 2
- net /LED4: track 0.00 -> 60.6 mm, vias 0 -> 2
- net /LED3: track 0.00 -> 59.2 mm, vias 0 -> 1
- net /RESET: track 0.00 -> 51.5 mm, vias 0 -> 1
- net /INT1: track 0.00 -> 43.1 mm
- net /RX: track 0.00 -> 43.1 mm, vias 0 -> 2
- net /TX: track 0.00 -> 35.0 mm, vias 0 -> 2
- net Net-(J4-Pad1): track 0.00 -> 24.5 mm
- net /LED5: track 0.00 -> 20.2 mm
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- added copper zone on B.Cu, net GND
- added copper zone on F.Cu, net GND
Other:
- net class Default: trace_width 0.25 -> 0.4; via_dia 0.6 -> 1.5; via_drill 0.4 -> 1

Commit message: Trena Rev 1
Signed-off-by: cuki2 <mauricio@krebs.com.br>
Parts:
- added J6: HC-SR04, w_pin_strip:pin_socket_4, F.Cu at (24.4, 49.8)
Connections:
- U1 pad 7: /XTAL2 -> /XTAL1
- U1 pad 8: /XTAL1 -> /XTAL2
Routing:
- net /INT2: track 73.1 -> 126.4 mm
- net Net-(J5-Pad1): track 6.48 -> 12.9 mm
- net +5V: track 254.9 -> 258.6 mm
- net /XTAL2: track 12.3 -> 15.3 mm
- net /XTAL1: track 11.9 -> 8.88 mm

Commit message: Rev 2 Trena
Signed-off-by: cuki2 <mauricio@krebs.com.br>
Parts:
- moved C2 7.88 mm to (35.3, 67.8), turned to 90 degrees
- moved C5 7.62 mm to (35.3, 75.2), turned to 270 degrees
- moved Q3 1.02 mm to (68.1, 44.7), turned to 180 degrees
- moved R12 0.76 mm to (71.9, 45.7)
- moved R13 0.76 mm to (71.9, 43.2)
- turned Y1 to 270 degrees
Routing:
- net +5V: track 258.6 -> 292.1 mm
- net GND: track 159.2 -> 191.9 mm, vias 8 -> 10
- net /INT2: track 126.4 -> 115.1 mm
- net Net-(Q3-Pad1): track 10.9 -> 2.10 mm
- net /RX: track 43.1 -> 49.0 mm, vias 2 -> 4
- net /XTAL1: track 8.88 -> 12.5 mm
- net /XTAL2: track 15.3 -> 12.1 mm
- net Net-(J4-Pad1): track 24.5 -> 26.8 mm, vias 0 -> 1

Commit message: Trena Posicionamento REV 3
Signed-off-by: cuki2 <mauricio@krebs.com.br>
Parts:
- removed J2: ICSP, w_pin_strip:pin_strip_3x2
- removed J4: IN, w_pin_strip:pin_socket_2
- D4: value TX -> LED_3; footprint w_smd_leds:Led_0805 -> w_indicators:led_3mm_clear
- D5: value RX -> PWR
- D6: value LED_3 -> RX; footprint w_indicators:led_3mm_clear -> w_smd_leds:Led_0805
- D7: value PWR -> TX
- J1: value RJ45 -> ICSP; footprint w_conn_pc:rj45-shield -> w_pin_strip:pin_strip_3x2
- J5: value OUT -> HC-SR04; footprint w_pin_strip:pin_socket_2 -> w_pin_strip:pin_socket_4
- J6: value HC-SR04 -> RJ45; footprint w_pin_strip:pin_socket_4 -> w_conn_pc:rj45-shield
- R10: value 360R -> 560R
- R11: value 360R -> 10k
- R12, R19: value 10k -> 560R
- R13: value 1k -> 360R
- R14: value 10k -> 360R
- R15, R9: value 560R -> 10k
- R16, R7: value 560R -> 1k
- R17: value 120R -> 10k
- R18: value 120R -> 560R
- R20, R4: value 1k -> 120R
- R8: value 10k -> 1k
- moved R17 60.4 mm to (23.9, 37.3), turned to 180 degrees
- moved R9 53.3 mm to (24.4, 47.0)
- moved R7 52.1 mm to (29.2, 46.0), turned to 270 degrees
- moved R19 49.0 mm to (35.1, 34.3), turned to 180 degrees
- moved C10 48.8 mm to (30.7, 34.3), turned to 0 degrees
- moved R14 48.8 mm to (23.9, 39.4), turned to 0 degrees
- moved R13 48.6 mm to (23.9, 35.3), turned to 0 degrees
- moved D5 48.2 mm to (53.3, 22.1), turned to 180 degrees
- moved U3 47.0 mm to (30.7, 38.1)
- moved R18 46.4 mm to (35.1, 41.7)
- moved J1 44.7 mm to (34.8, 63.8)
- moved R5 44.7 mm to (58.2, 22.1)
- moved C3 44.6 mm to (26.9, 47.0), turned to 270 degrees
- moved D6 43.9 mm to (43.7, 40.4), turned to 0 degrees
- moved Q1 43.7 mm to (25.9, 42.9), turned to 90 degrees
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Connections:
- D4 pad 1: /TX -> Net-(D4-Pad1)
- D4 pad 2: Net-(D4-Pad2) -> /LED5
- D5 pad 2: Net-(D5-Pad2) -> +5V
- D6 pad 2: /LED5 -> Net-(D6-Pad2)
- D7 pad 1: Net-(D7-Pad1) -> /TX
- D7 pad 2: +5V -> Net-(D7-Pad2)
- J1 pad 1: GND -> /MISO
- J1 pad 2: /PIN -> +5V
- J1 pad 3: Net-(J1-Pad3) -> /SCK
- J1 pad 4: /A -> /MOSI
- J1 pad 5: /B -> /RESET
- J1 pad 6: Net-(J1-Pad6) -> GND
- J5 pad 1: Net-(J5-Pad1) -> +5V
- J5 pad 2: GND -> Net-(J4-Pad1)
- J6 pad 1: +5V -> GND
- J6 pad 2: Net-(J5-Pad1) -> /PIN
- J6 pad 3: /INT2 -> Net-(J6-Pad3)
- J6 pad 4: GND -> /A
- Q2 pad 2: Net-(J5-Pad1) -> Net-(J4-Pad1)
- R10 pad 1: Net-(D5-Pad1) -> Net-(D6-Pad2)
- R10 pad 2: /RX -> +5V
- R11 pad 1: Net-(R11-Pad1) -> +5V
- R11 pad 2: /TX -> Net-(J4-Pad1)
- R12 pad 2: /INT2 -> Net-(D7-Pad2)
- R13 pad 1: Net-(Q3-Pad1) -> Net-(D6-Pad1)
- R13 pad 2: Net-(J4-Pad1) -> /RX
- R14 pad 1: +5V -> Net-(R14-Pad1)
- R14 pad 2: Net-(D5-Pad1) -> /TX
- R15 pad 1: /A -> +5V
- R15 pad 2: +5V -> /INT2
- R16 pad 1: GND -> Net-(Q3-Pad1)
- R16 pad 2: /B -> Net-(J3-Pad1)
- R17 pad 1: /B -> +5V
- R17 pad 2: /A -> Net-(D6-Pad1)
- R18 pad 1: Net-(D6-Pad1) -> /A
- R18 pad 2: /LED6 -> +5V
- R19 pad 1: /TX -> GND
- R19 pad 2: +5V -> /B
- R20 pad 1: GND -> /B
- R20 pad 2: Net-(D7-Pad1) -> /A
- R4 pad 1: /TX -> Net-(D4-Pad1)
- R4 pad 2: Net-(Q1-Pad1) -> /LED6
- R5 pad 1: Net-(Q2-Pad1) -> GND
- R5 pad 2: /INT1 -> Net-(D5-Pad1)
- R6 pad 1: +5V -> /TX
- R6 pad 2: Net-(Q1-Pad2) -> +5V
- R7 pad 1: Net-(D5-Pad2) -> /TX
- R7 pad 2: +5V -> Net-(Q1-Pad1)
- R8 pad 1: +5V -> Net-(Q2-Pad1)
- R8 pad 2: Net-(J5-Pad1) -> /INT1
- R9 pad 2: Net-(D4-Pad2) -> Net-(Q1-Pad2)
- U3 pad 1: Net-(D5-Pad1) -> Net-(D6-Pad1)
- U3 pad 4: Net-(R11-Pad1) -> Net-(R14-Pad1)
Routing:
- net +5V: track 292.1 -> 0.00 mm, vias 4 -> 0
- net GND: track 191.9 -> 0.00 mm, vias 10 -> 0
- net /INT2: track 115.1 -> 0.00 mm, vias 2 -> 0
- net /LED1: track 85.0 -> 0.00 mm, vias 1 -> 0
- net /A: track 72.7 -> 0.00 mm, vias 3 -> 0
- net /B: track 71.9 -> 0.00 mm, vias 1 -> 0
- net /LED2: track 61.0 -> 0.00 mm, vias 2 -> 0
- net /LED4: track 60.6 -> 0.00 mm, vias 2 -> 0
- net /LED3: track 59.2 -> 0.00 mm, vias 1 -> 0
- net /RESET: track 51.5 -> 0.00 mm, vias 1 -> 0
- net /RX: track 49.0 -> 0.00 mm, vias 4 -> 0
- net /INT1: track 43.1 -> 0.00 mm
- net /TX: track 35.0 -> 0.00 mm, vias 2 -> 0
- net Net-(J4-Pad1): track 26.8 -> 0.00 mm, vias 1 -> 0
- net /LED5: track 20.2 -> 0.00 mm
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Other:
- board size 70.7 x 70.7 mm -> 41 x 60 mm

Commit message: Trema Rev 3
Signed-off-by: cuki2 <mauricio@krebs.com.br>
Parts:
- added D10: LED_3, w_indicators:led_3mm_clear, F.Cu at (17.8, 52.3)
- added D8: LED1, w_indicators:led_3mm_clear, F.Cu at (17.8, 47.5)
- added D9: LED_2, w_indicators:led_3mm_clear, F.Cu at (17.8, 42.7)
- added Q4: BC817-40, w_smd_trans:sot23, F.Cu at (17.5, 38.1)
- added Q5: BC817-40, w_smd_trans:sot23, F.Cu at (51.1, 47.5)
- added R21: 1k, w_smd_resistors:r_0805, F.Cu at (48.0, 47.5)
- D2: value LED1 -> LED VERDE
- D3: value LED_2 -> LED VERDE
- D4: value LED_3 -> LED VERDE
- R2, R4: value 120R -> 10k
- R3: value 120R -> 1k
- moved R3 38.2 mm to (17.5, 34.5)
- moved R4 32.7 mm to (17.8, 56.4), turned to 180 degrees
- moved D2 13.5 mm to (56.6, 47.5)
- moved R2 8.32 mm to (56.6, 56.6)
- moved J5 7.55 mm to (48.0, 65.0)
- moved Q2 7.54 mm to (46.5, 58.7), turned to 0 degrees
- moved R11 6.82 mm to (45.5, 62.2)
- moved Q3 6.43 mm to (52.8, 61.0), turned to 0 degrees
- moved R16 6.37 mm to (49.3, 61.2)
- moved R15 6.19 mm to (56.6, 62.0), turned to 270 degrees
- moved D4 6.18 mm to (56.6, 42.7)
- moved R19 4.10 mm to (38.9, 35.8), turned to 90 degrees
- moved C10 4.06 mm to (34.8, 34.3), turned to 180 degrees
- moved D3 2.74 mm to (56.6, 52.3)
- moved R8 1.63 mm to (41.4, 60.7), turned to 0 degrees
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Connections:
- D2 pad 2: /LED1 -> +5V
- D3 pad 1: Net-(D3-Pad1) -> Net-(D2-Pad1)
- D3 pad 2: /LED3 -> +5V
- D4 pad 1: Net-(D4-Pad1) -> Net-(D2-Pad1)
- D4 pad 2: /LED5 -> +5V
- R2 pad 1: Net-(D2-Pad1) -> +5V
- R2 pad 2: /LED2 -> Net-(D2-Pad1)
- R3 pad 1: Net-(D3-Pad1) -> /LED2
- R3 pad 2: /LED4 -> Net-(Q4-Pad1)
- R4 pad 1: Net-(D4-Pad1) -> +5V
- R4 pad 2: /LED6 -> Net-(D10-Pad1)
- U1 pad 25: /LED3 -> Net-(U1-Pad25)
- U1 pad 26: /LED4 -> Net-(U1-Pad26)
- U1 pad 27: /LED5 -> Net-(U1-Pad27)
- U1 pad 28: /LED6 -> Net-(U1-Pad28)
Routing:
- net +5V: track 0.00 -> 269.0 mm, vias 0 -> 8
- net GND: track 0.00 -> 104.7 mm, vias 0 -> 3
- net /LED2: track 0.00 -> 57.7 mm, vias 0 -> 2
- net /PIN: track 0.00 -> 45.6 mm
- net /TX: track 0.00 -> 37.2 mm, vias 0 -> 3
- net /RX: track 0.00 -> 33.1 mm, vias 0 -> 2
- net /RESET: track 0.00 -> 27.8 mm, vias 0 -> 1
- net /INT2: track 0.00 -> 26.4 mm, vias 0 -> 2
- net /INT1: track 0.00 -> 25.0 mm, vias 0 -> 2
- net Net-(D6-Pad1): track 0.00 -> 24.3 mm, vias 0 -> 2
- net /SCK: track 0.00 -> 19.7 mm
- net Net-(C6-Pad1): track 0.00 -> 19.4 mm
- net Net-(D10-Pad1): track 0.00 -> 18.4 mm
- net Net-(D2-Pad1): track 0.00 -> 17.4 mm
- net /A: track 0.00 -> 17.3 mm
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Other:
- board size 41 x 60 mm -> 47 x 47 mm
- net class Default: clearance 0.2 -> 0.1; trace_width 0.4 -> 0.25
- net class PWR added: clearance 0.2, trace_width 0.4, via_dia 1.5, via_drill 1
- rule trace_clearance: 0.2 -> 0.1

Commit message: trena trafo ee16 lnk364pn
Signed-off-by: cuki <mauriciocukier@gmail.com>
Parts:
- D10: value LED_3 -> LED VERDE; footprint w_indicators:led_3mm_clear -> LEDs:LED_0805
- D2: footprint w_indicators:led_3mm_clear -> LEDs:LED_0805
- D3, D4: value LED VERDE -> LED VERMELHO; footprint w_indicators:led_3mm_clear -> LEDs:LED_0805
- D8: value LED1 -> LED VERMELHO; footprint w_indicators:led_3mm_clear -> LEDs:LED_0805
- D9: value LED_2 -> LED VERDE; footprint w_indicators:led_3mm_clear -> LEDs:LED_0805
- moved D4 40.1 mm to (17.3, 50.0), turned to 180 degrees
- moved D3 39.7 mm to (17.3, 47.5), turned to 180 degrees
- moved D9 39.6 mm to (56.6, 50.0), turned to 0 degrees
- moved D10 38.9 mm to (56.6, 52.3), turned to 0 degrees
- moved D8 4.85 mm to (17.3, 52.3), turned to 180 degrees
- turned D2 to 0 degrees
Connections:
- D2 pad 1: Net-(D2-Pad1) -> Net-(D10-Pad1)
- D3 pad 1: Net-(D2-Pad1) -> Net-(D3-Pad1)
- D4 pad 1: Net-(D2-Pad1) -> Net-(D3-Pad1)
- D8 pad 1: Net-(D10-Pad1) -> Net-(D3-Pad1)
- Q4 pad 2: Net-(D10-Pad1) -> Net-(D3-Pad1)
- Q5 pad 2: Net-(D2-Pad1) -> Net-(D10-Pad1)
- R2 pad 2: Net-(D2-Pad1) -> Net-(D10-Pad1)
- R4 pad 2: Net-(D10-Pad1) -> Net-(D3-Pad1)
Routing:
- net Net-(D3-Pad1): track 0.00 -> 18.9 mm
- net +5V: track 269.0 -> 287.8 mm, vias 8 -> 9
- net Net-(D2-Pad1): track 17.4 -> 0.00 mm
- net Net-(D10-Pad1): track 18.4 -> 13.1 mm
