File: Trena/sch/Trena.kicad_pcb (KiCad board)
At the start: 2 copper layers, 47 x 47 mm, 54 parts, among them J1 ICSP, J5 HC-SR04, J6 RJ45, Q1 PN2222A, Q2 BC817-40, Q3 BC817-40, Q4 BC817-40, Q5 BC817-40, U1 ATMEGA328P-AU, U2 LM1117-5.0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

Commit message: BOM Trena
Signed-off-by: maurice <mauricio@krebs.com.br>
Parts:
- D10: value LED_3 -> LED VERDE; footprint w_indicators:led_3mm_clear -> w_smd_leds:Led_0805
- D2: footprint w_indicators:led_3mm_clear -> w_smd_leds:Led_0805
- D3, D4: value LED VERDE -> LED VERMELHO; footprint w_indicators:led_3mm_clear -> w_smd_leds:Led_0805
- D8: value LED1 -> LED VERMELHO; footprint w_indicators:led_3mm_clear -> w_smd_leds:Led_0805
- D9: value LED_2 -> LED VERDE; footprint w_indicators:led_3mm_clear -> w_smd_leds:Led_0805
- moved D3 40.0 mm to (17.8, 42.7), turned to 180 degrees
- moved D4 39.1 mm to (17.8, 47.0), turned to 180 degrees
- moved D9 38.8 mm to (56.4, 47.0), turned to 0 degrees
- moved D10 38.6 mm to (56.4, 51.3), turned to 0 degrees
- moved D2 4.83 mm to (56.4, 42.7), turned to 0 degrees
- moved D8 3.81 mm to (17.8, 51.3), turned to 180 degrees
- moved R2 0.25 mm to (56.4, 56.6)
Connections:
- D2 pad 1: Net-(D2-Pad1) -> Net-(D10-Pad1)
- D3 pad 1: Net-(D2-Pad1) -> Net-(D3-Pad1)
- D4 pad 1: Net-(D2-Pad1) -> Net-(D3-Pad1)
- D8 pad 1: Net-(D10-Pad1) -> Net-(D3-Pad1)
- Q4 pad 2: Net-(D10-Pad1) -> Net-(D3-Pad1)
- Q5 pad 2: Net-(D2-Pad1) -> Net-(D10-Pad1)
- R2 pad 2: Net-(D2-Pad1) -> Net-(D10-Pad1)
- R4 pad 2: Net-(D10-Pad1) -> Net-(D3-Pad1)
Routing:
- net +5V: track 269.0 -> 242.9 mm, vias 8 -> 10
- net Net-(D3-Pad1): track 0.00 -> 18.8 mm
- net Net-(D2-Pad1): track 17.4 -> 0.00 mm
- net /INT1: track 25.0 -> 22.7 mm
- net /PIN: track 45.6 -> 43.6 mm
