File: Trena/sch/Trena.sch (KiCad schematic (older format))
At the start: 52 parts, among them J1 ICSP, J2 SL1, J3 IN, J4 OUT, J5 HC-SR04, J6 RJ45, Q1 PN2222A, Q2 BC817-40, Q3 BC817-40, Q4 BC817-40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

Commit message: trena trafo ee16 lnk364pn
Signed-off-by: cuki <mauriciocukier@gmail.com>
Parts:
- removed D1: D_ALT, w_smd_diode:do219ab, symbol D_ALT
- removed F1: Polyfuse, w_smd_resistors:r_1210, symbol Polyfuse
- added 250V: V250LA20CP, Varistors:RV_Disc_D21.5_W4.3_P10, symbol Varistor
- added C?: 100n, Capacitors_SMD:C_0805, symbol C
- added D? (x2): LED VERDE, LEDs:LED_0805, symbol LED_ALT
- added D? (x3): LED VERMELHO, LEDs:LED_0805, symbol LED_ALT
- added D?: D_Bridge_+-AA, symbol D_Bridge_+-AA
- added D?: D_Zener, symbol D_Zener
- added J?: IN, symbol Conn_01x02
- added R?: 390R, Resistors_SMD:R_0805, symbol R
- added R?: 1k, Resistors_SMD:R_0805, symbol R
- added TR?: TEZ6.0-D-2, Transformers_THT:Transformer_Breve_TEZ-38x45, symbol TEZ6.0-D-2
- added U?: LNK362P, Power_Integrations:PDIP-8B, symbol LNK362P
- added U?: PC817, Housings_DIP:DIP-4_W7.62mm, symbol PC817
- C?: renamed from C6; value 470uF -> 3.3uF 250V; footprint w_capacitors:CP_8x11.5mm -> Capacitors_THT:CP_Axial_L11.0mm_D8.0mm_P15.00mm_Horizontal
- C?: renamed from C7; footprint w_smd_cap:c_0805 -> Capacitors_SMD:C_0805
- C?: renamed from C8; footprint w_smd_cap:c_0805 -> Capacitors_SMD:C_0805
- C?: renamed from C9; footprint w_capacitors:CP_5x7mm -> Capacitors_THT:CP_Axial_L11.0mm_D5.0mm_P18.00mm_Horizontal
- C?: renamed from C4; footprint w_smd_cap:c_0805 -> Capacitors_SMD:C_0805
- C?: renamed from C3; footprint w_smd_cap:c_0805 -> Capacitors_SMD:C_0805
- C?: renamed from C1; footprint w_smd_cap:c_0805 -> Capacitors_SMD:C_0805
- C?: renamed from C2; footprint w_smd_cap:c_0805 -> Capacitors_SMD:C_0805
- C?: renamed from C5; footprint w_smd_cap:c_0805 -> Capacitors_SMD:C_0805
- C?: renamed from C10; footprint w_smd_cap:c_0805 -> Capacitors_SMD:C_0805
- D?: renamed from D2; footprint w_smd_leds:Led_0805 -> LEDs:LED_0805
- D?: renamed from D7; footprint w_smd_leds:Led_0805 -> LEDs:LED_0805
- D?: renamed from D6; footprint w_smd_leds:Led_0805 -> LEDs:LED_0805
- D?: renamed from D5; footprint w_smd_leds:Led_0805 -> LEDs:LED_0805
- J?: renamed from J1; footprint w_pin_strip:pin_strip_3x2 -> Pin_Headers:Pin_Header_Straight_2x03_Pitch2.54mm
- J?: renamed from J2; footprint w_pin_strip:pin_socket_2 -> Socket_Strips:Socket_Strip_Straight_1x02_Pitch2.54mm
- J?: renamed from J4; footprint w_pin_strip:pin_socket_2 -> Socket_Strips:Socket_Strip_Straight_1x02_Pitch2.54mm
- J?: renamed from J3; footprint w_pin_strip:pin_socket_2 -> Socket_Strips:Socket_Strip_Straight_1x02_Pitch2.54mm
- J?: renamed from J6; footprint w_conn_pc:rj45-shield -> Connectors:RJ45_8
- J?: renamed from J5; footprint w_pin_strip:pin_socket_4 -> Socket_Strips:Socket_Strip_Straight_1x04_Pitch2.54mm
- Q?: renamed from Q2; footprint w_smd_trans:sot23 -> TO_SOT_Packages_SMD:TSOT-23
- Q?: renamed from Q1; footprint w_smd_trans:sot23 -> TO_SOT_Packages_SMD:TSOT-23
- Q?: renamed from Q3; footprint w_smd_trans:sot23 -> TO_SOT_Packages_SMD:TSOT-23
- Q?: renamed from Q5; footprint w_smd_trans:sot23 -> TO_SOT_Packages_SMD:TSOT-23
- Q?: renamed from Q4; footprint w_smd_trans:sot23 -> TO_SOT_Packages_SMD:TSOT-23
- R?: renamed from R1; footprint w_smd_resistors:r_0805 -> Resistors_SMD:R_0805
- R?: renamed from R8; footprint w_smd_resistors:r_0805 -> Resistors_SMD:R_0805
- R?: renamed from R11; footprint w_smd_resistors:r_0805 -> Resistors_SMD:R_0805
- R?: renamed from R16; footprint w_smd_resistors:r_0805 -> Resistors_SMD:R_0805
- R?: renamed from R15; footprint w_smd_resistors:r_0805 -> Resistors_SMD:R_0805
- R?: renamed from R7; footprint w_smd_resistors:r_0805 -> Resistors_SMD:R_0805
- R?: renamed from R9; footprint w_smd_resistors:r_0805 -> Resistors_SMD:R_0805
- R?: renamed from R13; footprint w_smd_resistors:r_0805 -> Resistors_SMD:R_0805
- R?: renamed from R14; footprint w_smd_resistors:r_0805 -> Resistors_SMD:R_0805
- R?: renamed from R18; footprint w_smd_resistors:r_0805 -> Resistors_SMD:R_0805
- R?: renamed from R20; footprint w_smd_resistors:r_0805 -> Resistors_SMD:R_0805
- R?: renamed from R19; footprint w_smd_resistors:r_0805 -> Resistors_SMD:R_0805
- R?: renamed from R2; footprint w_smd_resistors:r_0805 -> Resistors_SMD:R_0805
- R?: renamed from R10; footprint w_smd_resistors:r_0805 -> Resistors_SMD:R_0805
- R?: renamed from R17; footprint w_smd_resistors:r_0805 -> Resistors_SMD:R_0805
- R?: renamed from R12; footprint w_smd_resistors:r_0805 -> Resistors_SMD:R_0805
- R?: renamed from R6; footprint w_smd_resistors:r_0805 -> Resistors_SMD:R_0805
- R?: renamed from R5; footprint w_smd_resistors:r_0805 -> Resistors_SMD:R_0805
- R?: renamed from R21; footprint w_smd_resistors:r_0805 -> Resistors_SMD:R_0805
- R?: renamed from R3; footprint w_smd_resistors:r_0805 -> Resistors_SMD:R_0805
- R?: renamed from R4; footprint w_smd_resistors:r_0805 -> Resistors_SMD:R_0805
- U?: renamed from U1; footprint w_smd_lqfp:lqfp32 -> Housings_QFP:TQFP-32_7x7mm_Pitch0.8mm
- U?: renamed from U2; footprint w_smd_trans:sot223 -> TO_SOT_Packages_SMD:SOT-223; symbol LM1117-5.0 -> LM1117-5.0-RESCUE-Trena
- U?: renamed from U3; footprint w_smd_dil:so-8 -> Housings_SOIC:SOIC-8_3.9x4.9mm_Pitch1.27mm
- Y?: renamed from Y1; footprint w_crystal:crystal_hc-49%2fsmd -> Crystals:Crystal_SMD_HC49-SD
Connections:
- net labels removed: PIN
- wire segments 165 -> 211
- no-connect marks 19 -> 20
Other:
- moved on the sheet: C?, D?, J?, Q?, R?, U?, Y?
