File: Trena/sch/Trena.sch (KiCad schematic (older format))
At the start: 50 parts, among them J1 RJ45, J2 ICSP, J3 SL1, J4 IN, J5 OUT, Q1 PN2222A, Q2 BC817-40, Q3 BC817-40, U1 ATMEGA328P-AU, U2 LM1117-5.0, U3 SP3485CN, Y1 Crystal

Commit message: Trena Rev 1
Signed-off-by: cuki2 <mauricio@krebs.com.br>
Parts:
- added J6: HC-SR04, w_pin_strip:pin_socket_4, symbol CONN_01X04
Connections:
- net +5V: now also J6.1 (P1)
- net GND: now also J6.4 (P4)
- net INT2: now also J6.3 (P3)
- net at J5.1 (P1), Q2.2 (C), R8.2: now also J6.2 (P2)
- no-connect marks 14 -> 15
Changed lines of the file:
@@
 LIBS:contrib
 LIBS:valves
+LIBS:Trena-cache
 EELAYER 25 0
 EELAYER END
@@
 Sheet 1 1
 Title "Trena Serial"
-Date "2017-12-19"
-Rev "0"
+Date "2018-01-31"
+Rev "1"
 Comp ""
 Comment1 "Mauricio Cukier"
@@
 	7950 2800 7950 2750
 Wire Wire Line
-	7450 2800 7950 2800
+	7450 2800 8200 2800
 Wire Wire Line
 	7700 2800 7700 2850
@@
 B
 $Comp
-L GND #PWR40
+L GND #PWR42
 U 1 1 5A3EA008
 P 9750 2100
-F 0 "#PWR40" H 9750 1850 50  0001 C CNN
+F 0 "#PWR42" H 9750 1850 50  0001 C CNN
 F 1 "GND" H 9750 1950 50  0000 C CNN
 F 2 "" H 9750 2100 50  0001 C CNN
@@
 Wire Wire Line
 	6500 800  6500 900
+$Comp
+L CONN_01X04 J6
+U 1 1 5A71B6EF
+P 9600 2800
+F 0 "J6" H 9600 3050 50  0000 C CNN
+F 1 "HC-SR04" V 9700 2800 50  0000 C CNN
+F 2 "w_pin_strip:pin_socket_4" H 9600 2800 50  0001 C CNN
+F 3 "" H 9600 2800 50  0001 C CNN
+	1    9600 2800
+	1    0    0    -1
+$EndComp
+$Comp
+L +5V #PWR40
+U 1 1 5A71BA6C
+P 9300 2600
+F 0 "#PWR40" H 9300 2450 50  0001 C CNN
+F 1 "+5V" H 9300 2740 50  0000 C CNN
+F 2 "" H 9300 2600 50  0001 C CNN
+F 3 "" H 9300 2600 50  0001 C CNN
+	1    9300 2600
+	1    0    0    -1
+$EndComp
+Wire Wire Line
+	9300 2600 9300 2650
+Wire Wire Line
+	9300 2650 9400 2650
+Wire Wire Line
+	9400 2750 8350 2750
+Wire Wire Line
+	8350 2750 8350 1900
+Connection ~ 8350 1900
+Wire Wire Line
+	8200 2800 8200 2850
+Wire Wire Line
+	8200 2850 9400 2850
+Connection ~ 7950 2800
+$Comp
+L GND #PWR41
+U 1 1 5A71BE32
+P 9300 3050
+F 0 "#PWR41" H 9300 2800 50  0001 C CNN
+F 1 "GND" H 9300 2900 50  0000 C CNN
+F 2 "" H 9300 3050 50  0001 C CNN
+F 3 "" H 9300 3050 50  0001 C CNN
+	1    9300 3050
+	1    0    0    -1
+$EndComp
+Wire Wire Line
+	9300 3050 9300 2950
+Wire Wire Line
+	9300 2950 9400 2950
+NoConn ~ 10650 1200
 $EndSCHEMATC

Commit message: Trena Posicionamento REV 3
Signed-off-by: cuki2 <mauricio@krebs.com.br>
Parts:
- renumbered D6 to D4, D7 to D5, D5 to D6, D4 to D7, J2 to J1, J3 to J2, J4 to J3, J5 to J4, J6 to J5, J1 to J6, R7 to R10, R8 to R11, R9 to R12, R10 to R13, R11 to R14, R12 to R15, R13 to R16, R14 to R17, R15 to R18, R16 to R19, R17 to R20, R18 to R4, R20 to R5, R19 to R6, R4 to R7, R5 to R8, R6 to R9
Connections:
- net INT2: no longer J5.3 (P3)
- net at J3.1 (P1), R16.2: now also J5.3 (P3)
Changed lines of the file:
@@
 Sheet 1 1
 Title "Trena Serial"
-Date "2018-02-02"
-Rev "2"
+Date "2018-02-05"
+Rev "3"
 Comp ""
 Comment1 "Mauricio Cukier"
@@
 XTAL2
 $Comp
-L CONN_02X03 J2
+L CONN_02X03 J1
 U 1 1 5A39C28D
 P 2550 5200
-F 0 "J2" H 2550 5400 50  0000 C CNN
+F 0 "J1" H 2550 5400 50  0000 C CNN
 F 1 "ICSP" H 2550 5000 50  0000 C CNN
 F 2 "w_pin_strip:pin_strip_3x2" H 2550 4000 50  0001 C CNN
@@
 $EndComp
 $Comp
-L R R5
+L R R8
 U 1 1 5A3A137E
 P 7150 2150
-F 0 "R5" V 7230 2150 50  0000 C CNN
+F 0 "R8" V 7230 2150 50  0000 C CNN
 F 1 "1k" V 7150 2150 50  0000 C CNN
 F 2 "w_smd_resistors:r_0805" V 7080 2150 50  0001 C CNN
@@
 	7700 2450 7700 2350
 $Comp
-L R R8
+L R R11
 U 1 1 5A3A19E2
 P 7700 1650
-F 0 "R8" V 7780 1650 50  0000 C CNN
+F 0 "R11" V 7780 1650 50  0000 C CNN
 F 1 "10k" V 7700 1650 50  0000 C CNN
 F 2 "w_smd_resistors:r_0805" V 7630 1650 50  0001 C CNN
@@
 $EndComp
 $Comp
-L R R13
+L R R16
 U 1 1 5A3A5332
 P 8250 3050
-F 0 "R13" V 8330 3050 50  0000 C CNN
+F 0 "R16" V 8330 3050 50  0000 C CNN
 F 1 "1k" V 8250 3050 50  0000 C CNN
 F 2 "w_smd_resistors:r_0805" V 8180 3050 50  0001 C CNN
@@
 	7700 3350 7700 3250
 $Comp
-L R R12
+L R R15
 U 1 1 5A3A553A
 P 7950 2600
-F 0 "R12" V 8030 2600 50  0000 C CNN
+F 0 "R15" V 8030 2600 50  0000 C CNN
 F 1 "10k" V 7950 2600 50  0000 C CNN
 F 2 "w_smd_resistors:r_0805" V 7880 2600 50  0001 C CNN
@@
 	1    0    0    -1
 $EndComp
-Wire Wire Line
-	7950 2800 7950 2750
-Wire Wire Line
-	7450 2800 8200 2800
-Wire Wire Line
-	7700 2800 7700 2850
 $Comp
 L +5V #PWR023
@@
 Wire Wire Line
 	7950 2400 7950 2450
-Connection ~ 7700 2800
 Text Label 7450 2800 0    60   ~ 0
 INT2
 $Comp
-L R R4
+L R R7
 U 1 1 5A3A7361
 P 6800 5400
-F 0 "R4" V 6880 5400 50  0000 C CNN
+F 0 "R7" V 6880 5400 50  0000 C CNN
 F 1 "1k" V 6800 5400 50  0000 C CNN
 F 2 "w_smd_resistors:r_0805" V 6730 5400 50  0001 C CNN
@@
 	7350 5650 7350 5600
 $Comp
-L R R6
+L R R9
 U 1 1 5A3A808C
 P 7350 4950
-F 0 "R6" V 7430 4950 50  0000 C CNN
+F 0 "R9" V 7430 4950 50  0000 C CNN
 F 1 "10k" V 7350 4950 50  0000 C CNN
 F 2 "w_smd_resistors:r_0805" V 7280 4950 50  0001 C CNN
@@
 Connection ~ 8000 5150
 $Comp
-L R R10
+L R R13
 U 1 1 5A3A93CB
 P 7850 4850
-F 0 "R10" V 7930 4850 50  0000 C CNN
+F 0 "R13" V 7930 4850 50  0000 C CNN
 F 1 "360R" V 7850 4850 50  0000 C CNN
 F 2 "w_smd_resistors:r_0805" V 7780 4850 50  0001 C CNN
@@
 	8000 4850 8100 4850
 $Comp
-L R R11
+L R R14
 U 1 1 5A3A9C03
 P 7850 5250
-F 0 "R11" V 7930 5250 50  0000 C CNN
+F 0 "R14" V 7930 5250 50  0000 C CNN
 F 1 "360R" V 7850 5250 50  0000 C CNN
 F 2 "w_smd_resistors:r_0805" V 7780 5250 50  0001 C CNN
@@
 	8900 3750 8900 3700
 $Comp
-L R R15
+L R R18
 U 1 1 5A3AFED2
 P 9250 4650
-F 0 "R15" V 9330 4650 50  0000 C CNN
+F 0 "R18" V 9330 4650 50  0000 C CNN
 F 1 "560R" V 9250 4650 50  0000 C CNN
 F 2 "w_smd_resistors:r_0805" V 9180 4650 50  0001 C CNN
@@
 	9250 4400 9250 4500
 $Comp
-L R R17
+L R R20
 U 1 1 5A3B096E
 P 9550 5050
-F 0 "R17" V 9630 5050 50  0000 C CNN
+F 0 "R20" V 9630 5050 50  0000 C CNN
 F 1 "120R" V 9550 5050 50  0000 C CNN
 F 2 "w_smd_resistors:r_0805" V 9480 5050 50  0001 C CNN
@@
 	9400 5150 8900 5150
 $Comp
-L R R16
+L R R19
 U 1 1 5A3B0BE8
 P 9250 5400
-F 0 "R16" V 9330 5400 50  0000 C CNN
+F 0 "R19" V 9330 5400 50  0000 C CNN
 F 1 "560R" V 9250 5400 50  0000 C CNN
 F 2 "w_smd_resistors:r_0805" V 9180 5400 50  0001 C CNN
@@
 B
 $Comp
-L CONN_01X02 J3
+L CONN_01X02 J2
 U 1 1 5A3B174A
 P 8000 4350
-F 0 "J3" H 8000 4500 50  0000 C CNN
+F 0 "J2" H 8000 4500 50  0000 C CNN
 F 1 "SL1" V 8100 4350 50  0000 C CNN
 F 2 "w_pin_strip:pin_socket_2" H 8000 4350 50  0001 C CNN
@@
 	8600 3050 8400 3050
 $Comp
-L CONN_01X02 J5
+L CONN_01X02 J4
 U 1 1 5A3B5C2C
 P 8850 1950
-F 0 "J5" H 8850 2100 50  0000 C CNN
+F 0 "J4" H 8850 2100 50  0000 C CNN
 F 1 "OUT" V 8950 1950 50  0000 C CNN
 F 2 "w_pin_strip:pin_socket_2" H 8850 1950 50  0001 C CNN
@@
 	8550 2000 8650 2000
 $Comp
-L CONN_01X02 J4
+L CONN_01X02 J3
 U 1 1 5A3B719C
 P 8800 3100
-F 0 "J4" H 8800 3250 50  0000 C CNN
+F 0 "J3" H 8800 3250 50  0000 C CNN
 F 1 "IN" V 8900 3100 50  0000 C CNN
 F 2 "w_pin_strip:pin_socket_2" H 8800 3100 50  0001 C CNN
@@
 	5600 6100 5350 6100
 $Comp
-L LED_ALT D4
+L LED_ALT D7
 U 1 1 5A3C2E43
 P 8050 5700
-F 0 "D4" H 8050 5800 50  0000 C CNN
+F 0 "D7" H 8050 5800 50  0000 C CNN
 F 1 "TX" H 8050 5600 50  0000 C CNN
 F 2 "w_smd_leds:Led_0805" H 8050 5700 50  0001 C CNN
@@
 	7450 4600 8300 4600
 $Comp
-L R R7
+L R R10
 U 1 1 5A3C3DB6
 P 7450 3900
-F 0 "R7" V 7530 3900 50  0000 C CNN
+F 0 "R10" V 7530 3900 50  0000 C CNN
 F 1 "560R" V 7450 3900 50  0000 C CNN
 F 2 "w_smd_resistors:r_0805" V 7380 3900 50  0001 C CNN
@@
 	7450 4050 7450 4150
 $Comp
-L R R14
+L R R17
 U 1 1 5A3C4726
 P 8300 4200
-F 0 "R14" V 8380 4200 50  0000 C CNN
+F 0 "R17" V 8380 4200 50  0000 C CNN
 F 1 "10k" V 8300 4200 50  0000 C CNN
 F 2 "w_smd_resistors:r_0805" V 8230 4200 50  0001 C CNN
@@
 	8300 3950 8300 4050
 $Comp
-L LED_ALT D5
+L LED_ALT D6
 U 1 1 5A3C639E
 P 7450 4300
-F 0 "D5" H 7450 4400 50  0000 C CNN
+F 0 "D6" H 7450 4400 50  0000 C CNN
 F 1 "RX" H 7450 4200 50  0000 C CNN
 F 2 "w_smd_leds:Led_0805" H 7450 4300 50  0001 C CNN
@@
 $EndComp
 $Comp
-L R R9
+L R R12
 U 1 1 5A3C7384
 P 7750 5900
-F 0 "R9" V 7830 5900 50  0000 C CNN
+F 0 "R12" V 7830 5900 50  0000 C CNN
 F 1 "560R" V 7750 5900 50  0000 C CNN
 F 2 "w_smd_resistors:r_0805" V 7680 5900 50  0001 C CNN
@@
 LED6
 $Comp
-L LED_ALT D6
+L LED_ALT D4
 U 1 1 5A3D8898
 P 4800 6450
-F 0 "D6" H 4800 6550 50  0000 C CNN
+F 0 "D4" H 4800 6550 50  0000 C CNN
 F 1 "LED_3" H 4800 6350 50  0000 C CNN
 F 2 "w_indicators:led_3mm_clear" H 4800 6450 50  0001 C CNN
@@
 $EndComp
 $Comp
-L R R18
+L R R4
 U 1 1 5A3D889E
 P 5200 6450
-F 0 "R18" V 5280 6450 50  0000 C CNN
+F 0 "R4" V 5280 6450 50  0000 C CNN
 F 1 "120R" V 5200 6450 50  0000 C CNN
 F 2 "w_smd_resistors:r_0805" V 5130 6450 50  0001 C CNN
@@
 Connection ~ 7650 5250
 $Comp
-L R R19
+L R R6
 U 1 1 5A3E46B2
 P 6600 5000
-F 0 "R19" V 6680 5000 50  0000 C CNN
+F 0 "R6" V 6680 5000 50  0000 C CNN
 F 1 "10k" V 6600 5000 50  0000 C CNN
 F 2 "w_smd_resistors:r_0805" V 6530 5000 50  0001 C CNN
@@
 Connection ~ 6550 5400
 $Comp
-L RJ45 J1
+L RJ45 J6
 U 1 1 5A3E658B
 P 10100 1550
-F 0 "J1" H 10300 2050 50  0000 C CNN
+F 0 "J6" H 10300 2050 50  0000 C CNN
 F 1 "RJ45" H 9950 2050 50  0000 C CNN
 F 2 "w_conn_pc:rj45-shield" H 10100 1550 50  0001 C CNN
@@
 NoConn ~ 10450 2000
 $Comp
-L LED_ALT D7
+L LED_ALT D5
 U 1 1 5A3ED0FC
 P 6500 1050
-F 0 "D7" H 6500 1150 50  0000 C CNN
+F 0 "D5" H 6500 1150 50  0000 C CNN
 F 1 "PWR" H 6500 950 50  0000 C CNN
 F 2 "w_smd_leds:Led_0805" H 6500 1050 50  0001 C CNN
@@
 $EndComp
 $Comp
-L R R20
+L R R5
 U 1 1 5A3EE5AB
 P 6500 1450
-F 0 "R20" V 6580 1450 50  0000 C CNN
+F 0 "R5" V 6580 1450 50  0000 C CNN
 F 1 "1k" V 6500 1450 50  0000 C CNN
 F 2 "w_smd_resistors:r_0805" V 6430 1450 50  0001 C CNN
@@
 	6500 800  6500 900
 $Comp
-L CONN_01X04 J6
+L CONN_01X04 J5
 U 1 1 5A71B6EF
 P 9600 2800
-F 0 "J6" H 9600 3050 50  0000 C CNN
+F 0 "J5" H 9600 3050 50  0000 C CNN
 F 1 "HC-SR04" V 9700 2800 50  0000 C CNN
 F 2 "w_pin_strip:pin_socket_4" H 9600 2800 50  0001 C CNN
@@
 	8350 2750 8350 1900
 Connection ~ 8350 1900
-Wire Wire Line
-	8200 2800 8200 2850
-Wire Wire Line
-	8200 2850 9400 2850
-Connection ~ 7950 2800
 $Comp
 L GND #PWR042
@@
 	9300 2950 9400 2950
 NoConn ~ 10650 1200
+Wire Wire Line
+	7450 2800 7950 2800
+Wire Wire Line
+	7950 2800 7950 2750
+Wire Wire Line
+	7700 2850 7700 2800
+Connection ~ 7700 2800
+Wire Wire Line
+	9400 2850 8500 2850
+Wire Wire Line
+	8500 2850 8500 3050
+Connection ~ 8500 3050
 $EndSCHEMATC

Commit message: Trema Rev 3
Signed-off-by: cuki2 <mauricio@krebs.com.br>
Parts:
- removed D3: LED_2, w_indicators:led_3mm_clear, symbol LED_ALT
- removed D4: LED_3, w_indicators:led_3mm_clear, symbol LED_ALT
- added Q4, Q5: BC817-40, w_smd_trans:sot23, symbol Q_NPN_BCE
- added R21: 1k, w_smd_resistors:r_0805, symbol R
- D2: value LED1 -> LED VERDE; footprint w_indicators:led_3mm_clear -> w_smd_leds:Led_0805
- R2, R4: value 120R -> 10k
- R3: value 120R -> 1k
Connections:
- net labels removed: LED3, LED4, LED5, LED6
- wire segments 150 -> 165
- no-connect marks 15 -> 19
Other:
- moved on the sheet: D2, R2

Commit message: BOM Trena
Signed-off-by: maurice <mauricio@krebs.com.br>
Parts:
- removed J2: SL1, w_pin_strip:pin_socket_2, symbol CONN_01X02
- removed J3: IN, w_pin_strip:pin_socket_2, symbol CONN_01X02
- removed J4: OUT, w_pin_strip:pin_socket_2, symbol CONN_01X02
- added D10, D8, D9: LED VERDE, w_smd_leds:Led_0805, symbol LED_ALT
- added D3, D4: LED VERMELHO, w_smd_leds:Led_0805, symbol LED_ALT
- C1, C10, C3, C4, C7, C8: Desc (none) -> capacitor ceramico smd 0805
- C2, C5: Desc (none) -> capacitor ceramico 22pF smd 0805
- C6: Desc (none) -> capacitor eletrolitico 470uF 25V
- C9: Desc (none) -> capacitor eletrolitico 470uF 6V
- D1: Desc (none) -> diodo 1n4007 smd do-214aac (smb)
- D2: value LED VERDE -> LED VERMELHO; Desc (none) -> led vermelho smd 0805
- D5: Desc (none) -> led verde smd 0805
- D6: Desc (none) -> led vermelho smd 0805
- D7: Desc (none) -> led azul smd 0805
- F1: value Polyfuse -> 500ma; Desc (none) -> fusivel rapido 500ma 63v smd 1206
- J1: Desc (none) -> barra de pinos 2x3 vias
- J5: Desc (none) -> barra de pinos 1x4 vias
- J6: Desc (none) -> conector RJ45 90 graus
- Q1: Desc (none) -> transistor npn 2n2222 smd sot23
- Q2, Q3, Q4, Q5: Desc (none) -> transistor npn bc817-25 smd sot23
- R1, R17, R2, R4, R6, R9: Desc (none) -> resisotor 10k smd 0805
- R10, R12: value 560R -> 10k; Desc (none) -> resisotor 10k smd 0805
- R11: value 10k -> 560R; Desc (none) -> resisotor 560R smd 0805
- R13: Desc (none) -> resisotor 360R smd 0805
- R14: value 360R -> 560R; Desc (none) -> resisotor 560R smd 0805
- R15: value 10k -> 360R; Desc (none) -> resisotor 360R smd 0805
- R16, R21, R3, R5, R7, R8: Desc (none) -> resisotor 1k smd 0805
- R18, R19: Desc (none) -> resisotor 560R smd 0805
- R20: Desc (none) -> resisotor 120R smd 0805
- U1: Desc (none) -> microcontrolador atmega328p smd qfp32
- U2: symbol LM1117-5.0 -> LM1117-5.0-RESCUE-Trena; Desc (none) -> regulador de tensao lm1117-5.0 smd sot223
- U3: Desc (none) -> circuito integrado max485 smd so-8
- Y1: Desc (none) -> cristal 16MHz smd hc-49sm
Connections:
- wire segments 165 -> 157
Other:
- moved on the sheet: C1, C2, C5, C6, C9, D1, D6, D7, F1, J1, J5, J6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
